File: windlogger_shield/kicad_files/F1 Anemometre.sch (KiCad schematic (older format))
At the start: 22 parts, among them U201 LMV358

Commit message: Add files
Parts:
- C201, C202, C203: symbol C -> C-RESCUE-Windlogger
- R201, R202, R203, R204, R205, R206, R207, R208, R209, R210: symbol R -> R-RESCUE-Windlogger
Changed lines of the file:
@@
 EESchema Schematic File Version 2
+LIBS:Windlogger-rescue
 LIBS:power
 LIBS:device
@@
 LIBS:memory
 LIBS:xilinx
-LIBS:special
 LIBS:microcontrollers
 LIBS:dsp
@@
 LIBS:valves
 LIBS:Windlogger-cache
-EELAYER 27 0
+EELAYER 25 0
 EELAYER END
 $Descr A4 11693 8268
@@
 Wind2
 $Comp
-L R R203
+L R-RESCUE-Windlogger R203
 U 1 1 56137C0A
 P 3750 4850
@@
 $EndComp
 $Comp
-L +3.3V #PWR015
+L +3.3V-RESCUE-Windlogger #PWR015
 U 1 1 56137D24
 P 6450 4850
+AR Path="/56137D24" Ref="#PWR015"  Part="1"
+AR Path="/560A35D3/56137D24" Ref="#PWR015"  Part="1"
 F 0 "#PWR015" H 6450 4810 30  0001 C CNN
 F 1 "+3.3V" H 6450 4960 30  0000 C CNN
@@
 	7050 5400 7750 5400
 $Comp
-L R R208
+L R-RESCUE-Windlogger R208
 U 1 1 56137DBB
 P 5950 6700
@@
 $EndComp
 $Comp
-L R R210
+L R-RESCUE-Windlogger R210
 U 1 1 56137DCA
 P 6450 6300
@@
 Speed2
 $Comp
-L +3.3V #PWR018
+L +3.3V-RESCUE-Windlogger #PWR018
 U 1 1 56137E91
 P 8700 3950
+AR Path="/56137E91" Ref="#PWR018"  Part="1"
+AR Path="/560A35D3/56137E91" Ref="#PWR018"  Part="1"
 F 0 "#PWR018" H 8700 3910 30  0001 C CNN
 F 1 "+3.3V" H 8700 4060 30  0000 C CNN
@@
 $EndComp
 $Comp
-L C C203
+L C-RESCUE-Windlogger C203
 U 1 1 56137EA0
 P 8700 4300
@@
 $EndComp
 $Comp
-L +3.3V #PWR020
+L +3.3V-RESCUE-Windlogger #PWR020
 U 1 1 56137F32
 P 5300 2000
+AR Path="/56137F32" Ref="#PWR020"  Part="1"
+AR Path="/560A35D3/56137F32" Ref="#PWR020"  Part="1"
 F 0 "#PWR020" H 5300 1960 30  0001 C CNN
 F 1 "+3.3V" H 5300 2110 30  0000 C CNN
@@
 $EndComp
 $Comp
-L R R209
+L R-RESCUE-Windlogger R209
 U 1 1 56137926
 P 6300 3400
@@
 $EndComp
 $Comp
-L R R207
+L R-RESCUE-Windlogger R207
 U 1 1 5613790D
 P 5750 3750
@@
 $EndComp
 $Comp
-L +3.3V #PWR023
+L +3.3V-RESCUE-Windlogger #PWR023
 U 1 1 56137563
 P 6250 1800
+AR Path="/56137563" Ref="#PWR023"  Part="1"
+AR Path="/560A35D3/56137563" Ref="#PWR023"  Part="1"
 F 0 "#PWR023" H 6250 1760 30  0001 C CNN
 F 1 "+3.3V" H 6250 1910 30  0000 C CNN
@@
 $EndComp
 $Comp
-L C C201
+L C-RESCUE-Windlogger C201
 U 1 1 561373CB
 P 4350 1800
@@
 $EndComp
 $Comp
-L R R201
+L R-RESCUE-Windlogger R201
 U 1 1 561373BC
 P 3700 1900
@@
 	3700 1500 4950 1500
 $Comp
-L R R205
+L R-RESCUE-Windlogger R205
 U 1 1 5614E4FA
 P 4350 3250
@@
 $EndComp
 $Comp
-L +3.3V #PWR026
+L +3.3V-RESCUE-Windlogger #PWR026
 U 1 1 5614E500
 P 4350 2700
+AR Path="/5614E500" Ref="#PWR026"  Part="1"
+AR Path="/560A35D3/5614E500" Ref="#PWR026"  Part="1"
 F 0 "#PWR026" H 4350 2660 30  0001 C CNN
 F 1 "+3.3V" H 4350 2810 30  0000 C CNN
@@
 $EndComp
 $Comp
-L +3.3V #PWR027
+L +3.3V-RESCUE-Windlogger #PWR027
 U 1 1 5614E6DA
 P 5300 4950
+AR Path="/5614E6DA" Ref="#PWR027"  Part="1"
+AR Path="/560A35D3/5614E6DA" Ref="#PWR027"  Part="1"
 F 0 "#PWR027" H 5300 4910 30  0001 C CNN
 F 1 "+3.3V" H 5300 5060 30  0000 C CNN
@@
 $EndComp
 $Comp
-L C C202
+L C-RESCUE-Windlogger C202
 U 1 1 5614E6FE
 P 4400 5100
@@
 Connection ~ 4400 4450
 $Comp
-L R R206
+L R-RESCUE-Windlogger R206
 U 1 1 5614E70E
 P 4400 6300
@@
 $EndComp
 $Comp
-L +3.3V #PWR030
+L +3.3V-RESCUE-Windlogger #PWR030
 U 1 1 5614E714
 P 4400 5650
+AR Path="/5614E714" Ref="#PWR030"  Part="1"
+AR Path="/560A35D3/5614E714" Ref="#PWR030"  Part="1"
 F 0 "#PWR030" H 4400 5610 30  0001 C CNN
 F 1 "+3.3V" H 4400 5760 30  0000 C CNN
@@
 	3700 2300 3700 2150
 $Comp
-L R R202
+L R-RESCUE-Windlogger R202
 U 1 1 561FBC5D
 P 3700 3150
@@
 	3700 3400 3700 3550
 $Comp
-L R R204
+L R-RESCUE-Windlogger R204
 U 1 1 561FBD15
 P 3750 6150
