File: windlogger_shield/kicad_files/F2 Girouette.sch (KiCad schematic (older format))
At the start: 8 parts, among them U301 LMV358

Commit message: Add files
Parts:
- C301, C302: symbol C -> C-RESCUE-Windlogger
- R301, R302, R303: symbol R -> R-RESCUE-Windlogger
Changed lines of the file:
@@
 EESchema Schematic File Version 2
+LIBS:Windlogger-rescue
 LIBS:power
 LIBS:device
@@
 LIBS:memory
 LIBS:xilinx
-LIBS:special
 LIBS:microcontrollers
 LIBS:dsp
@@
 LIBS:valves
 LIBS:Windlogger-cache
-EELAYER 27 0
+EELAYER 25 0
 EELAYER END
 $Descr A4 11693 8268
@@
 $EndDescr
 $Comp
-L R R301
+L R-RESCUE-Windlogger R301
 U 1 1 561261A3
 P 4400 2550
@@
 $EndComp
 $Comp
-L C C301
+L C-RESCUE-Windlogger C301
 U 1 1 561264FC
 P 5700 3900
@@
 $EndComp
 $Comp
-L +3.3V #PWR033
+L +3.3V-RESCUE-Windlogger #PWR033
 U 1 1 561265CA
 P 7300 2850
+AR Path="/561265CA" Ref="#PWR033"  Part="1"
+AR Path="/560A35DE/561265CA" Ref="#PWR033"  Part="1"
 F 0 "#PWR033" H 7300 2810 30  0001 C CNN
 F 1 "+3.3V" H 7300 2960 30  0000 C CNN
@@
 vane_sig
 $Comp
-L +3.3V #PWR034
+L +3.3V-RESCUE-Windlogger #PWR034
 U 1 1 56126B28
 P 8850 4000
+AR Path="/56126B28" Ref="#PWR034"  Part="1"
+AR Path="/560A35DE/56126B28" Ref="#PWR034"  Part="1"
 F 0 "#PWR034" H 8850 3960 30  0001 C CNN
 F 1 "+3.3V" H 8850 4110 30  0000 C CNN
@@
 $EndComp
 $Comp
-L C C302
+L C-RESCUE-Windlogger C302
 U 1 1 56126B37
 P 8850 4400
@@
 	8850 4600 8850 4800
 $Comp
-L R R302
+L R-RESCUE-Windlogger R302
 U 1 1 5612799B
 P 5150 3300
@@
 	3550 2900 4400 2900
 $Comp
-L +3.3V #PWR036
+L +3.3V-RESCUE-Windlogger #PWR036
 U 1 1 561389E2
 P 4400 2150
+AR Path="/561389E2" Ref="#PWR036"  Part="1"
+AR Path="/560A35DE/561389E2" Ref="#PWR036"  Part="1"
 F 0 "#PWR036" H 4400 2110 30  0001 C CNN
 F 1 "+3.3V" H 4400 2260 30  0000 C CNN
@@
 	6800 3500 6800 4150
 $Comp
-L R R303
+L R-RESCUE-Windlogger R303
 U 1 1 561FBEB5
 P 7600 4150
@@
 $EndComp
 $Comp
-L +3.3V #PWR038
+L +3.3V-RESCUE-Windlogger #PWR038
 U 1 1 561FC307
 P 6300 2600
+AR Path="/561FC307" Ref="#PWR038"  Part="1"
+AR Path="/560A35DE/561FC307" Ref="#PWR038"  Part="1"
 F 0 "#PWR038" H 6300 2560 30  0001 C CNN
 F 1 "+3.3V" H 6300 2710 30  0000 C CNN
