File: windlogger_shield/kicad_files/F3 Wattmetre_ACsch.sch (KiCad schematic (older format))
At the start: 17 parts, among them U401 LMV358

Commit message: Add files
Parts:
- C401, C402, C403: symbol C -> C-RESCUE-Windlogger
- R401, R402, R403, R404, R405, R407, R408, R409: symbol R -> R-RESCUE-Windlogger
Changed lines of the file:
@@
 EESchema Schematic File Version 2
+LIBS:Windlogger-rescue
 LIBS:power
 LIBS:device
@@
 LIBS:memory
 LIBS:xilinx
-LIBS:special
 LIBS:microcontrollers
 LIBS:dsp
@@
 LIBS:valves
 LIBS:Windlogger-cache
-EELAYER 27 0
+EELAYER 25 0
 EELAYER END
 $Descr A4 11693 8268
@@
 $EndDescr
 $Comp
-L R R407
+L R-RESCUE-Windlogger R407
 U 1 1 561274B6
 P 7700 3800
@@
 $EndComp
 $Comp
-L R R408
+L R-RESCUE-Windlogger R408
 U 1 1 561274C5
 P 8300 3050
@@
 $EndComp
 $Comp
-L R R409
+L R-RESCUE-Windlogger R409
 U 1 1 561274D4
 P 8300 4500
@@
 $EndComp
 $Comp
-L C C402
+L C-RESCUE-Windlogger C402
 U 1 1 561274E3
 P 7700 4550
@@
 $EndComp
 $Comp
-L +3.3V #PWR040
+L +3.3V-RESCUE-Windlogger #PWR040
 U 1 1 56127501
 P 8300 2500
+AR Path="/56127501" Ref="#PWR040"  Part="1"
+AR Path="/560A361A/56127501" Ref="#PWR040"  Part="1"
 F 0 "#PWR040" H 8300 2460 30  0001 C CNN
 F 1 "+3.3V" H 8300 2610 30  0000 C CNN
@@
 $EndComp
 $Comp
-L +3.3V #PWR042
+L +3.3V-RESCUE-Windlogger #PWR042
 U 1 1 561275C6
 P 9650 2950
+AR Path="/561275C6" Ref="#PWR042"  Part="1"
+AR Path="/560A361A/561275C6" Ref="#PWR042"  Part="1"
 F 0 "#PWR042" H 9650 2910 30  0001 C CNN
 F 1 "+3.3V" H 9650 3060 30  0000 C CNN
@@
 UAC_lo
 $Comp
-L R R401
+L R-RESCUE-Windlogger R401
 U 1 1 56127660
 P 2800 4150
@@
 $EndComp
 $Comp
-L R R403
+L R-RESCUE-Windlogger R403
 U 1 1 5612766F
 P 3750 3700
@@
 $EndComp
 $Comp
-L R R404
+L R-RESCUE-Windlogger R404
 U 1 1 5612767E
 P 3750 5100
@@
 $EndComp
 $Comp
-L C C401
+L C-RESCUE-Windlogger C401
 U 1 1 5612768D
 P 3100 5100
@@
 $EndComp
 $Comp
-L +3.3V #PWR045
+L +3.3V-RESCUE-Windlogger #PWR045
 U 1 1 56127786
 P 3750 3000
+AR Path="/56127786" Ref="#PWR045"  Part="1"
+AR Path="/560A361A/56127786" Ref="#PWR045"  Part="1"
 F 0 "#PWR045" H 3750 2960 30  0001 C CNN
 F 1 "+3.3V" H 3750 3110 30  0000 C CNN
@@
 Connection ~ 7700 3400
 $Comp
-L +3.3V #PWR046
+L +3.3V-RESCUE-Windlogger #PWR046
 U 1 1 56128055
 P 5000 2700
+AR Path="/56128055" Ref="#PWR046"  Part="1"
+AR Path="/560A361A/56128055" Ref="#PWR046"  Part="1"
 F 0 "#PWR046" H 5000 2660 30  0001 C CNN
 F 1 "+3.3V" H 5000 2810 30  0000 C CNN
@@
 IAC
 $Comp
-L R R402
+L R-RESCUE-Windlogger R402
 U 1 1 56128120
 P 3400 4150
@@
 $EndComp
 $Comp
-L C C403
+L C-RESCUE-Windlogger C403
 U 1 1 561281A1
 P 8150 6350
@@
 $EndComp
 $Comp
-L +3.3V #PWR048
+L +3.3V-RESCUE-Windlogger #PWR048
 U 1 1 561283B2
 P 8150 5950
+AR Path="/561283B2" Ref="#PWR048"  Part="1"
+AR Path="/560A361A/561283B2" Ref="#PWR048"  Part="1"
 F 0 "#PWR048" H 8150 5910 30  0001 C CNN
 F 1 "+3.3V" H 8150 6060 30  0000 C CNN
@@
 	4500 3400 4500 4000
 $Comp
-L R R405
+L R-RESCUE-Windlogger R405
 U 1 1 561E1890
 P 7700 2850
@@
 $EndComp
 $Comp
-L +3.3V #PWR050
+L +3.3V-RESCUE-Windlogger #PWR050
 U 1 1 561FC074
 P 4250 2550
+AR Path="/561FC074" Ref="#PWR050"  Part="1"
+AR Path="/560A361A/561FC074" Ref="#PWR050"  Part="1"
 F 0 "#PWR050" H 4250 2510 30  0001 C CNN
 F 1 "+3.3V" H 4250 2660 30  0000 C CNN
@@
 $EndComp
 $Comp
-L +3.3V #PWR052
+L +3.3V-RESCUE-Windlogger #PWR052
 U 1 1 561FC1BD
 P 8750 2700
+AR Path="/561FC1BD" Ref="#PWR052"  Part="1"
+AR Path="/560A361A/561FC1BD" Ref="#PWR052"  Part="1"
 F 0 "#PWR052" H 8750 2660 30  0001 C CNN
 F 1 "+3.3V" H 8750 2810 30  0000 C CNN
