File: windlogger_shield/kicad_files/F4 Wattmetre_DC.sch (KiCad schematic (older format))
At the start: 7 parts, among them U301 LMV358

Commit message: Add files
Parts:
- R501, R503, R504: symbol R -> R-RESCUE-Windlogger
Changed lines of the file:
@@
 EESchema Schematic File Version 2
+LIBS:Windlogger-rescue
 LIBS:power
 LIBS:device
@@
 LIBS:memory
 LIBS:xilinx
-LIBS:special
 LIBS:microcontrollers
 LIBS:dsp
@@
 LIBS:valves
 LIBS:Windlogger-cache
-EELAYER 27 0
+EELAYER 25 0
 EELAYER END
 $Descr A4 11693 8268
@@
 UDC_hi
 $Comp
-L R R503
+L R-RESCUE-Windlogger R503
 U 1 1 561287F5
 P 4650 4800
@@
 $EndComp
 $Comp
-L +3.3V #PWR056
+L +3.3V-RESCUE-Windlogger #PWR056
 U 1 1 56128856
 P 6500 3950
+AR Path="/56128856" Ref="#PWR056"  Part="1"
+AR Path="/560A3643/56128856" Ref="#PWR056"  Part="1"
 F 0 "#PWR056" H 6500 3910 30  0001 C CNN
 F 1 "+3.3V" H 6500 4060 30  0000 C CNN
@@
 Use the jumper to select the maximum voltage :\n64V for Battery system\n640V to monitor a DC bus from an on grid system
 $Comp
-L R R501
+L R-RESCUE-Windlogger R501
 U 1 1 561E1CF9
 P 4300 3850
@@
 $EndComp
 $Comp
-L R R504
+L R-RESCUE-Windlogger R504
 U 1 1 561E1D08
 P 5000 3850
@@
 $EndComp
 $Comp
-L +3.3V #PWR057
+L +3.3V-RESCUE-Windlogger #PWR057
 U 1 1 561FC3A0
 P 5500 3700
+AR Path="/561FC3A0" Ref="#PWR057"  Part="1"
+AR Path="/560A3643/561FC3A0" Ref="#PWR057"  Part="1"
 F 0 "#PWR057" H 5500 3660 30  0001 C CNN
 F 1 "+3.3V" H 5500 3810 30  0000 C CNN
