File: windlogger_shield/kicad_files/F5 Temperature.sch (KiCad schematic (older format))
At the start: 9 parts, among them U701 LMV358

Commit message: Add files
Parts:
- C701: symbol C -> C-RESCUE-Windlogger
- R701, R702, R703, R704, R705, R706: symbol R -> R-RESCUE-Windlogger
Changed lines of the file:
@@
 EESchema Schematic File Version 2
+LIBS:Windlogger-rescue
 LIBS:power
 LIBS:device
@@
 LIBS:memory
 LIBS:xilinx
-LIBS:special
 LIBS:microcontrollers
 LIBS:dsp
@@
 LIBS:valves
 LIBS:Windlogger-cache
-EELAYER 27 0
+EELAYER 25 0
 EELAYER END
 $Descr A4 11693 8268
@@
 $EndComp
 $Comp
-L +3.3V #PWR070
+L +3.3V-RESCUE-Windlogger #PWR070
 U 1 1 561521EF
 P 4100 2600
+AR Path="/561521EF" Ref="#PWR070"  Part="1"
+AR Path="/560A36CB/561521EF" Ref="#PWR070"  Part="1"
 F 0 "#PWR070" H 4100 2560 30  0001 C CNN
 F 1 "+3.3V" H 4100 2710 30  0000 C CNN
@@
 $EndComp
 $Comp
-L +3.3V #PWR073
+L +3.3V-RESCUE-Windlogger #PWR073
 U 1 1 561522F5
 P 5900 3150
+AR Path="/561522F5" Ref="#PWR073"  Part="1"
+AR Path="/560A36CB/561522F5" Ref="#PWR073"  Part="1"
 F 0 "#PWR073" H 5900 3110 30  0001 C CNN
 F 1 "+3.3V" H 5900 3260 30  0000 C CNN
@@
 Utemp
 $Comp
-L C C701
+L C-RESCUE-Windlogger C701
 U 1 1 5615255D
 P 7250 5500
@@
 $EndComp
 $Comp
-L +3.3V #PWR074
+L +3.3V-RESCUE-Windlogger #PWR074
 U 1 1 5615256C
 P 7250 5150
+AR Path="/5615256C" Ref="#PWR074"  Part="1"
+AR Path="/560A36CB/5615256C" Ref="#PWR074"  Part="1"
 F 0 "#PWR074" H 7250 5110 30  0001 C CNN
 F 1 "+3.3V" H 7250 5260 30  0000 C CNN
@@
 temp_lo
 $Comp
-L R R701
+L R-RESCUE-Windlogger R701
 U 1 1 561E1EE7
 P 4100 3000
@@
 $EndComp
 $Comp
-L R R703
+L R-RESCUE-Windlogger R703
 U 1 1 5624BBCD
 P 4100 4850
@@
 $EndComp
 $Comp
-L R R702
+L R-RESCUE-Windlogger R702
 U 1 1 562792A9
 P 5200 4250
@@
 $EndComp
 $Comp
-L R R704
+L R-RESCUE-Windlogger R704
 U 1 1 562792B8
 P 5900 4700
@@
 Connection ~ 6650 3700
 $Comp
-L R R705
+L R-RESCUE-Windlogger R705
 U 1 1 5627934E
 P 7300 3700
@@
 $EndComp
 $Comp
-L R R706
+L R-RESCUE-Windlogger R706
 U 1 1 562793BC
 P 8500 4700
@@
 	8500 3000 8500 3200
 $Comp
-L +3.3V #PWR077
+L +3.3V-RESCUE-Windlogger #PWR077
 U 1 1 56279444
 P 8500 3000
+AR Path="/56279444" Ref="#PWR077"  Part="1"
+AR Path="/560A36CB/56279444" Ref="#PWR077"  Part="1"
 F 0 "#PWR077" H 8500 2960 30  0001 C CNN
 F 1 "+3.3V" H 8500 3110 30  0000 C CNN
