File: windlogger_shield/kicad_files/F6 Alimentation.sch (KiCad schematic (older format))
At the start: 13 parts, among them SW601 SWITCH_INV, U601 LM2597M-3.3

Commit message: Add files
Parts:
- C602, C603, C605: symbol C -> C-RESCUE-Windlogger
- D603: symbol LED -> LED-RESCUE-Windlogger
- R605, R606: symbol R -> R-RESCUE-Windlogger
Changed lines of the file:
@@
 EESchema Schematic File Version 2
+LIBS:Windlogger-rescue
 LIBS:power
 LIBS:device
@@
 LIBS:memory
 LIBS:xilinx
-LIBS:special
 LIBS:microcontrollers
 LIBS:dsp
@@
 LIBS:valves
 LIBS:Windlogger-cache
-EELAYER 27 0
+EELAYER 25 0
 EELAYER END
 $Descr A4 11693 8268
@@
 NoConn ~ 2250 1700
 $Comp
-L C C603
+L C-RESCUE-Windlogger C603
 U 1 1 561F6D92
 P 6750 3450
@@
 $EndComp
 $Comp
-L C C602
+L C-RESCUE-Windlogger C602
 U 1 1 561F6D9F
 P 4650 3450
@@
 	9350 2900 9550 2900
 $Comp
-L R R605
+L R-RESCUE-Windlogger R605
 U 1 1 561F7977
 P 9800 2900
@@
 $EndComp
 $Comp
-L LED D603
+L LED-RESCUE-Windlogger D603
 U 1 1 561F797D
 P 10450 2900
@@
 Connection ~ 9350 2500
 $Comp
-L C C605
+L C-RESCUE-Windlogger C605
 U 1 1 561F99E6
 P 8900 2950
@@
 	8900 3150 8900 3400
 $Comp
-L R R606
+L R-RESCUE-Windlogger R606
 U 1 1 5624A22A
 P 4600 2200
@@
 Connection ~ 4600 2500
 $Comp
-L +3.3V #PWR067
+L +3.3V-RESCUE-Windlogger #PWR067
 U 1 1 56289455
 P 10100 2150
+AR Path="/56289455" Ref="#PWR067"  Part="1"
+AR Path="/560A36AF/56289455" Ref="#PWR067"  Part="1"
 F 0 "#PWR067" H 10100 2110 30  0001 C CNN
 F 1 "+3.3V" H 10100 2260 30  0000 C CNN
@@
 Connection ~ 4850 2900
 $Comp
-L +3.3V #PWR068
+L +3.3V-RESCUE-Windlogger #PWR068
 U 1 1 5630AD15
 P 4850 1700
+AR Path="/5630AD15" Ref="#PWR068"  Part="1"
+AR Path="/560A36AF/5630AD15" Ref="#PWR068"  Part="1"
 F 0 "#PWR068" H 4850 1660 30  0001 C CNN
 F 1 "+3.3V" H 4850 1810 30  0000 C CNN
@@
 $EndComp
 $Comp
-L +3.3V #PWR069
+L +3.3V-RESCUE-Windlogger #PWR069
 U 1 1 5630AD24
 P 4600 1700
+AR Path="/5630AD24" Ref="#PWR069"  Part="1"
+AR Path="/560A36AF/5630AD24" Ref="#PWR069"  Part="1"
 F 0 "#PWR069" H 4600 1660 30  0001 C CNN
 F 1 "+3.3V" H 4600 1810 30  0000 C CNN
