File: windlogger_shield/kicad_files/Windlogger.kicad_pcb (KiCad board)
At the start: 2 copper layers, 93.7 x 75.9 mm, 97 parts, among them K101 CONN_3, K102 CONN_3, P101 CONN_2, P102 CONN_5, P103 CONN_2, P104 CONN_2, P105 CONN_2, P106 CONN_2, P107 CONN_2, P108 CONN_2, P109 CONN_8, P110 CONN_6, P111 CONN_10, P112 CONN_8, P113 CONN_8, P114 CONN_6, P115 CONN_2, SW601 SWITCH_INV, U201 LMV358, U301 LMV358, U401 LMV358, U601 LM2597M-3.3, U701 LMV358

Commit message: Add files
Parts:
- added ?: VAL**, Trou_2_5_1_5, F.Cu at (95.1, 82.2)
- added ?: VAL**, Trou_2_5_1_5, F.Cu at (95.1, 132.3)
- added ?: VAL**, Trou_2_5_1_5, F.Cu at (95.1, 137.4)
- added ?: VAL**, Trou_2_5_1_5, F.Cu at (95.1, 86.6)
- added ?: VAL**, Trou_2_5_1_5, F.Cu at (95.1, 92.3)
- added ?: VAL**, Trou_2_5_1_5, F.Cu at (95.1, 97.4)
- added ?: VAL**, Trou_2_5_1_5, F.Cu at (95.1, 104.4)
- added ?: VAL**, Trou_2_5_1_5, F.Cu at (95.1, 109.5)
- added ?: VAL**, Trou_2_5_1_5, F.Cu at (95.1, 115.2)
- added ?: VAL**, Trou_2_5_1_5, F.Cu at (95.1, 120.3)
- added ?: VAL**, Trou_2_5_1_5, F.Cu at (95.1, 127.9)
- ? (x4): footprint Trou_3_10 -> lib:Trou_3_10
- C601, C604: footprint SMDHD/VF -> SMDHD_VF
- R403: value 45k -> 47k
- R701, R703: value 22.6k -> 20k
- moved D302 1.18 mm to (145.4, 116.8)
- moved D301 0.83 mm to (143.5, 113.7)
- moved R210 0.54 mm to (163.8, 104.8)
- moved R409 0.28 mm to (158.1, 131.5)
- moved P101 0.28 mm to (107.3, 135.3)
- moved ? 0.28 mm to (181.0, 81.9)
- moved C202 0.28 mm to (172.1, 104.8)
- moved C203 0.28 mm to (160.7, 95.9)
- moved C302 0.28 mm to (154.3, 111.1)
- moved C603 0.28 mm to (165.1, 81.9)
- moved C605 0.28 mm to (156.9, 81.9)
- moved C701 0.28 mm to (164.5, 111.1)
- moved D201 0.28 mm to (149.3, 102.2)
- moved D202 0.28 mm to (149.3, 97.2)
- moved D203 0.28 mm to (167.0, 97.7)
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Connections:
- P102 pad 2: (no net) -> Net-(P102-Pad2)
- P102 pad 3: (no net) -> Net-(P102-Pad3)
- P102 pad 4: (no net) -> Net-(P102-Pad4)
- P109 pad 1: (no net) -> Net-(P109-Pad1)
- P109 pad 2: (no net) -> Net-(P109-Pad2)
- P109 pad 3: (no net) -> Net-(P109-Pad3)
- P109 pad 8: (no net) -> Net-(P109-Pad8)
- P111 pad 1: (no net) -> Net-(P111-Pad1)
- P111 pad 10: (no net) -> Net-(P111-Pad10)
- P111 pad 2: (no net) -> Net-(P111-Pad2)
- P111 pad 3: (no net) -> Net-(P111-Pad3)
- P111 pad 5: (no net) -> Net-(P111-Pad5)
- P111 pad 6: (no net) -> Net-(P111-Pad6)
- P111 pad 7: (no net) -> Net-(P111-Pad7)
- P111 pad 8: (no net) -> Net-(P111-Pad8)
- P111 pad 9: (no net) -> Net-(P111-Pad9)
- P112 pad 5: (no net) -> Net-(P112-Pad5)
- P112 pad 6: (no net) -> Net-(P112-Pad6)
- P112 pad 7: (no net) -> Net-(P112-Pad7)
- P112 pad 8: (no net) -> Net-(P112-Pad8)
- P114 pad 1: (no net) -> Net-(P114-Pad1)
- SW601 pad 1: (no net) -> Net-(SW601-Pad1)
Routing:
- net /F6 Alimentation/Power_fail: track 87.6 -> 78.5 mm
- net Net-(P102-Pad2): track 0.00 -> 5.20 mm
- net AGND: track 544.7 -> 540.0 mm
- net /F5 Temperature/Utemp: track 68.6 -> 72.2 mm
- net /F1 Anemometre/Speed2: track 38.2 -> 35.2 mm, vias 2 -> 4
- net /F3 Wattmetre_AC/0-32A: track 15.5 -> 17.7 mm
- net /F4 Wattmetre_DC/UDC_hi: track 86.9 -> 88.3 mm
- net /F2 Girouette/vane_v+: track 38.2 -> 39.5 mm
- net +3.3V: track 331.7 -> 333.1 mm, vias 14 -> 13
- net /F3 Wattmetre_AC/IAC_hi: track 85.7 -> 87.0 mm
- net /F3 Wattmetre_AC/UAC_lo: track 86.0 -> 87.2 mm
- net Net-(R705-Pad2): track 21.2 -> 20.0 mm
- net Net-(C301-Pad1): track 13.5 -> 12.7 mm
- net Net-(R208-Pad1): track 6.48 -> 7.07 mm
- net /F5 Temperature/temp_lo: track 73.8 -> 73.2 mm
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- added copper zone on F.Cu, net Net-(C602-Pad1)
- removed copper zone on F.Cu, net N-0000070
Other:
- board size 93.7 x 75.9 mm -> 93.6 x 75.7 mm
- net class Windlogger: via_dia 0.415 -> 0.525; via_drill 0.245 -> 0.3
- rule trace_min: 0.05 -> 0.21
- rule via_min_drill: 0.208 -> 0.3
- rule via_min_size: 0.289 -> 0.525
- board text added: "Power supply"
