File: windlogger_shield/kicad_files/Windlogger.sch (KiCad schematic (older format))
At the start: 18 parts, among them K101 CONN_3, K102 CONN_3, P101 CONN_2, P102 CONN_5, P103 CONN_2, P104 CONN_2, P105 CONN_2, P106 CONN_2, P107 CONN_2, P108 CONN_2, P109 CONN_8, P110 CONN_6, P111 CONN_10, P112 CONN_8, P113 CONN_8, P114 CONN_6, P115 CONN_2

Commit message: Add files
Parts:
- R101: symbol R -> R-RESCUE-Windlogger
Changed lines of the file:
@@
 EESchema Schematic File Version 2
+LIBS:Windlogger-rescue
 LIBS:power
 LIBS:device
@@
 LIBS:memory
 LIBS:xilinx
-LIBS:special
 LIBS:microcontrollers
 LIBS:dsp
@@
 LIBS:valves
 LIBS:Windlogger-cache
-EELAYER 27 0
+EELAYER 25 0
 EELAYER END
 $Descr A4 11693 8268
@@
 IDC
 $Comp
-L +3.3V #PWR03
+L +3.3V-RESCUE-Windlogger #PWR03
 U 1 1 560A4057
 P 3200 4850
@@
 $EndComp
 $Comp
-L +3.3V #PWR07
+L +3.3V-RESCUE-Windlogger #PWR07
 U 1 1 560A5580
 P 8200 3000
@@
 NoConn ~ 9950 3600
 $Comp
-L R R101
+L R-RESCUE-Windlogger R101
 U 1 1 560B9C15
 P 1850 7050
@@
 $EndComp
 $Comp
-L +3.3V #PWR011
+L +3.3V-RESCUE-Windlogger #PWR011
 U 1 1 560B9C24
 P 1850 6700
