File: Hardware/shield/kicad/shield.kicad_pcb (KiCad board)
At the start: 2 copper layers, 135 x 95 mm, 110 parts, among them P101 anemo1, P102 anemo2, P103 vane, P104 AC_in, P105 DC_in, P106 current1, P107 current2, P108 current3, P109 current4, P110 temp, P111 RPM, P112 Power, P113 Analog, P114 5VDC, P115 POWER_SOURCE, P116 PWM, P117 PWM, P118 Communication, P119 h1, P120 h2, P121 h3, P122 h4, U201 LMV358, U301 LMV358, U401 LMV358, U501 LMV358, U502 LMV358, U601 LMV358

Commit message: add shield_preview.jpg
Parts:
- removed C101: CP, Capacitors_ThroughHole:C_Radial_D5_L6_P2.5
- removed C102: C, Capacitors_ThroughHole:C_Radial_D5_L6_P2.5
- removed C201, C202, C203, C301, C302, C401: 100nF, Capacitors_ThroughHole:C_Rect_L7_W2.5_P5
- removed C402, C501, C502, C503, C504: 10uF, Capacitors_ThroughHole:C_Radial_D5_L6_P2.5
- removed C601: 100nF, Capacitors_ThroughHole:C_Radial_D5_L6_P2.5
- removed D201, D202, D203, D204, D301, D302, D401, D402, D403, D404, D501, D502, D503, D504, D505, D506, D507, D508: 1N4148, Diodes_ThroughHole:Diode_DO-35_SOD27_Horizontal_RM10
- removed JP201, JP202, JP203, JP204, JP501, JP502, JP503, JP504: JUMPER3, Pin_Headers:Pin_Header_Straight_1x03
- removed NTC601: 2.2k, Discret:R4
- removed P119: h1, Socket_Arduino_Mega:Arduino_1pin
- removed R101, R204, R205, R404, R601, R602, R603, R604, R605, R606: 10k, Discret:R4
- removed R201, R202, R208, R209, R303, R403, R405, R406, R505, R506, R507, R508, R513, R514, R515, R516: 100k, Discret:R4
- removed R203, R301, R302: 100, Discret:R4
- removed R206, R207, R402: 1k, Discret:R4
- removed R401: 15k, Discret:R4
- removed R501, R502, R509, R510: 180, Discret:R4
- removed R503, R504, R511, R512: 90.9, Discret:R4
- removed U201, U301, U401, U501, U502, U601: LMV358, Housings_DIP:DIP-8_W7.62mm_LongPads
- added P123: h5, Socket_Arduino_Mega:Arduino_1pin, F.Cu at (83.4, 131.7)
- added P124: h6, Socket_Arduino_Mega:Arduino_1pin, F.Cu at (208.4, 131.7)
- added P125: h7, Socket_Arduino_Mega:Arduino_1pin, F.Cu at (83.4, 46.7)
- added P126: h8, Socket_Arduino_Mega:Arduino_1pin, F.Cu at (208.4, 46.7)
- moved P114 40.3 mm to (118.4, 46.7), turned to 180 degrees
- moved P104 11.0 mm to (98.4, 49.7)
- moved P106 10.0 mm to (139.4, 49.7)
- moved P107 10.0 mm to (160.4, 49.7)
- moved P108 10.0 mm to (181.4, 49.7)
- moved P109 10.0 mm to (202.4, 49.7)
- moved P115 9.00 mm to (105.4, 59.7)
- moved P105 7.00 mm to (109.4, 49.7)
Other:
- outline, holes or cut-outs redrawn
