File: Hardware/shield/kicad/shield.kicad_pcb (KiCad board)
At the start: 2 copper layers, 135 x 95 mm, 25 parts, among them P101 anemo1, P102 anemo2, P103 vane, P104 AC_in, P105 DC_in, P106 current1, P107 current2, P108 current3, P109 current4, P110 temp, P111 RPM, P112 Power, P113 Analog, P114 5VDC, P115 POWER_SOURCE, P116 PWM, P117 PWM, P118 Communication, P120 h2, P121 h3, P122 h4, P123 h5, P124 h6, P125 h7, P126 h8

Commit message: update digital files
Other:
- board text added: "AC IN"
- board text added: "Current1"
- board text added: "Current2"
- board text added: "Current3"
- board text added: "Current4"
- board text added: "DC IN"
- board text added: "RPM"
- board text added: "Temp"
- board text added: "Vane"
- board text added: "anemo1"
- board text added: "anemo2"
Changed lines of the file:
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@@
     (area 78.322539 41.617459 213.422541 136.717461)
     (thickness 1.6)
-    (drawings 8)
+    (drawings 19)
     (tracks 0)
     (zones 0)
@@
     (descr "Through hole socket strip")
     (tags "socket strip")
-    (fp_text reference P114 (at 0 -5.1 180) (layer F.SilkS)
+    (fp_text reference P114 (at 0.63 2.71 180) (layer F.SilkS)
       (effects (font (size 1 1) (thickness 0.15)))
     )
@@
     (descr "Through hole socket strip")
     (tags "socket strip")
-    (fp_text reference P115 (at 7 -5 360) (layer F.SilkS)
+    (fp_text reference P115 (at 11.43 0 360) (layer F.SilkS)
       (effects (font (size 1 1) (thickness 0.15)))
     )
@@
     (pad 1 thru_hole circle (at 0 0) (size 4.064 4.064) (drill 3.048) (layers *.Cu *.Mask F.SilkS))
   )
+  (gr_text Temp (at 197.75254 113.80746 90) (layer F.SilkS)
+    (effects (font (size 1.5 1.5) (thickness 0.3)))
+  )
+  (gr_text RPM (at 197.75254 102.37746 90) (layer F.SilkS)
+    (effects (font (size 1.5 1.5) (thickness 0.3)))
+  )
+  (gr_text Vane (at 197.75254 88.40746 90) (layer F.SilkS)
+    (effects (font (size 1.5 1.5) (thickness 0.3)))
+  )
+  (gr_text anemo2 (at 197.75254 75.70746 90) (layer F.SilkS)
+    (effects (font (size 1.5 1.5) (thickness 0.3)))
+  )
+  (gr_text anemo1 (at 197.75254 64.27746 90) (layer F.SilkS)
+    (effects (font (size 1.5 1.5) (thickness 0.3)))
+  )
+  (gr_text Current4 (at 193.94254 57.92746) (layer F.SilkS)
+    (effects (font (size 1.5 1.5) (thickness 0.3)))
+  )
+  (gr_text Current3 (at 173.62254 57.92746) (layer F.SilkS)
+    (effects (font (size 1.5 1.5) (thickness 0.3)))
+  )
+  (gr_text Current2 (at 152.03254 57.92746) (layer F.SilkS)
+    (effects (font (size 1.5 1.5) (thickness 0.3)))
+  )
+  (gr_text Current1 (at 131.71254 57.92746) (layer F.SilkS)
+    (effects (font (size 1.5 1.5) (thickness 0.3)))
+  )
+  (gr_text "DC IN" (at 106.31254 57.92746) (layer F.SilkS)
+    (effects (font (size 1.5 1.5) (thickness 0.3)))
+  )
+  (gr_text "AC IN" (at 96.15254 57.92746) (layer F.SilkS)
+    (effects (font (size 1.5 1.5) (thickness 0.3)))
+  )
   (gr_line (start 78.37254 44.16746) (end 78.37254 134.16746) (angle 90) (layer Edge.Cuts) (width 0.1))
