File: Hardware/digital/kicad/F1_output-a.sch (KiCad schematic (older format))
At the start: 18 parts, among them P201 SD CARD

Commit message: update digital files
Parts:
- P2001: renamed from P?; value CONN_02X04 -> WIFI; footprint (none) -> Socket_Strips:Socket_Strip_Straight_2x04
- P2002: renamed from P?; value CONN_01X07 -> GPRS; footprint (none) -> Socket_Strips:Socket_Strip_Straight_1x07
- P2003: renamed from P?; footprint (none) -> Socket_Strips:Socket_Strip_Straight_1x01
- U2001: renamed from U?; footprint (none) -> Housings_DIP:DIP-14_W7.62mm_LongPads
- U2002: renamed from U?; footprint (none) -> Hope_RFM:RFM69CW
Connections:
- net data_rx: now reaches U2001.11
- net data_tx: now reaches U2001.15
Other:
- note added: "ESP-01 or ESP-12 connector"
- note added: "M590E or A6 connector"
- note removed: "ESP-01 connector"
- note removed: "M590E connector"
- note removed: "rx"
- note removed: "tx"
Changed lines of the file:
@@
 $Descr A4 11693 8268
 encoding utf-8
-Sheet 2 2
+Sheet 2 3
 Title ""
 Date ""
@@
 SCLK
 Wire Wire Line
-	4850 2350 5150 2350
-Wire Wire Line
-	5150 2350 5850 2350
+	4850 2350 5850 2350
 Wire Wire Line
 	5700 2450 5850 2450
@@
 	5700 2750 6425 2750
 Wire Wire Line
-	4800 2850 4950 2850
-Wire Wire Line
-	4950 2850 6475 2850
-Wire Wire Line
-	5700 2450 5700 2750
-Wire Wire Line
-	5700 2750 5700 3150
+	4800 2850 6475 2850
+Wire Wire Line
+	5700 2450 5700 3150
 Wire Wire Line
 	5750 2550 5750 2050
@@
 $EndComp
 Wire Wire Line
-	4800 2250 5350 2250
-Wire Wire Line
-	5350 2250 5850 2250
+	4800 2250 5850 2250
 $Comp
 L R R202
@@
 Connection ~ 5150 2350
 Wire Wire Line
-	4950 1700 5150 1700
-Wire Wire Line
-	5150 1700 5350 1700
+	4950 1700 5350 1700
 Wire Wire Line
 	4950 1700 4950 1800
 Wire Wire Line
-	5150 1650 5150 1700
-Wire Wire Line
-	5150 1700 5150 1800
+	5150 1650 5150 1800
 Connection ~ 5150 1700
 Connection ~ 4950 2850
@@
 $EndComp
 $Comp
-L VAA #PWR204
+L VAA #PWR017
 U 1 1 5804B48D
 P 5750 2050
-F 0 "#PWR204" H 5750 2110 30  0001 C CNN
+F 0 "#PWR017" H 5750 2110 30  0001 C CNN
 F 1 "VAA" H 5750 2175 30  0000 C CNN
 F 2 "" H 5750 2050 60  0000 C CNN
@@
 	4500 2250 4425 2250
 Wire Wire Line
-	4425 2250 4425 2450
-Wire Wire Line
-	4425 2450 4425 2650
-Wire Wire Line
-	4425 2650 4425 2850
-Wire Wire Line
-	4425 2850 4425 3000
+	4425 2250 4425 3000
 Wire Wire Line
 	4425 2850 4500 2850
@@
 Connection ~ 4425 2450
 $Comp
-L GND #PWR201
+L GND #PWR018
 U 1 1 5804B49B
 P 4425 3000
-F 0 "#PWR201" H 4425 2750 50  0001 C CNN
+F 0 "#PWR018" H 4425 2750 50  0001 C CNN
 F 1 "GND" H 4425 2850 50  0000 C CNN
 F 2 "" H 4425 3000 50  0000 C CNN
@@
 $EndComp
 $Comp
-L +3.3V #PWR202
+L +3.3V #PWR019
 U 1 1 5804B4A1
 P 5150 1650
-F 0 "#PWR202" H 5150 1500 50  0001 C CNN
+F 0 "#PWR019" H 5150 1500 50  0001 C CNN
 F 1 "+3.3V" H 5150 1790 50  0000 C CNN
 F 2 "" H 5150 1650 50  0000 C CNN
@@
 $EndComp
 $Comp
-L GND #PWR203
+L GND #PWR020
 U 1 1 5804B4AE
 P 5700 3150
-F 0 "#PWR203" H 5700 2900 50  0001 C CNN
+F 0 "#PWR020" H 5700 2900 50  0001 C CNN
 F 1 "GND" H 5700 3000 50  0000 C CNN
 F 2 "" H 5700 3150 50  0000 C CNN
@@
 	6475 2550 6350 2550
 $Comp
-L 4050 U?
+L 4050 U2001
 U 1 1 5805ACEA
 P 2575 1400
-F 0 "U?" H 2770 1515 50  0000 C CNN
+F 0 "U2001" H 2770 1515 50  0000 C CNN
 F 1 "4050" H 2765 1275 50  0000 C CNN
-F 2 "" H 2575 1400 60  0000 C CNN
+F 2 "Housings_DIP:DIP-14_W7.62mm_LongPads" H 2575 1400 60  0001 C CNN
 F 3 "" H 2575 1400 60  0000 C CNN
 	1    2575 1400
@@
 $EndComp
 $Comp
-L 4050 U?
+L 4050 U2001
 U 2 1 5805AD41
 P 2575 1825
-F 0 "U?" H 2770 1940 50  0000 C CNN
+F 0 "U2001" H 2770 1940 50  0000 C CNN
 F 1 "4050" H 2765 1700 50  0000 C CNN
-F 2 "" H 2575 1825 60  0000 C CNN
+F 2 "Housings_DIP:DIP-14_W7.62mm_LongPads" H 2575 1825 60  0001 C CNN
 F 3 "" H 2575 1825 60  0000 C CNN
 	2    2575 1825
@@
 $EndComp
 $Comp
-L 4050 U?
+L 4050 U2001
 U 3 1 5805AD96
 P 2575 2225
-F 0 "U?" H 2770 2340 50  0000 C CNN
+F 0 "U2001" H 2770 2340 50  0000 C CNN
 F 1 "4050" H 2765 2100 50  0000 C CNN
-F 2 "" H 2575 2225 60  0000 C CNN
+F 2 "Housings_DIP:DIP-14_W7.62mm_LongPads" H 2575 2225 60  0001 C CNN
 F 3 "" H 2575 2225 60  0000 C CNN
 	3    2575 2225
@@
 $EndComp
 $Comp
-L 4050 U?
+L 4050 U2001
 U 4 1 5805ADD1
 P 2575 2625
-F 0 "U?" H 2770 2740 50  0000 C CNN
+F 0 "U2001" H 2770 2740 50  0000 C CNN
 F 1 "4050" H 2765 2500 50  0000 C CNN
-F 2 "" H 2575 2625 60  0000 C CNN
+F 2 "Housings_DIP:DIP-14_W7.62mm_LongPads" H 2575 2625 60  0001 C CNN
 F 3 "" H 2575 2625 60  0000 C CNN
 	4    2575 2625
@@
 $EndComp
 $Comp
-L 4050 U?
+L 4050 U2001
 U 5 1 5805AE0E
 P 2575 3200
-F 0 "U?" H 2770 3315 50  0000 C CNN
+F 0 "U2001" H 2770 3315 50  0000 C CNN
 F 1 "4050" H 2765 3075 50  0000 C CNN
-F 2 "" H 2575 3200 60  0000 C CNN
+F 2 "Housings_DIP:DIP-14_W7.62mm_LongPads" H 2575 3200 60  0001 C CNN
 F 3 "" H 2575 3200 60  0000 C CNN
 	5    2575 3200
@@
 $EndComp
 $Comp
-L 4050 U?
+L 4050 U2001
 U 6 1 5805AE51
 P 2575 3575
-F 0 "U?" H 2770 3690 50  0000 C CNN
+F 0 "U2001" H 2770 3690 50  0000 C CNN
 F 1 "4050" H 2765 3450 50  0000 C CNN
-F 2 "" H 2575 3575 60  0000 C CNN
+F 2 "Housings_DIP:DIP-14_W7.62mm_LongPads" H 2575 3575 60  0001 C CNN
 F 3 "" H 2575 3575 60  0000 C CNN
 	6    2575 3575
@@
 Wire Wire Line
 	1625 2625 2125 2625
-Text Notes 1925 3200 0    60   ~ 0
-rx
-Text Notes 1925 3600 0    60   ~ 0
-tx
 Text Notes 8975 1250 0    60   ~ 0
 rfm69cw in spi
@@
 SD card
 $Comp
-L RFM69CW U?
+L RFM69CW U2002
 U 1 1 5805B811
 P 9225 2375
-F 0 "U?" H 9225 1975 60  0000 C CNN
+F 0 "U2002" H 9225 1975 60  0000 C CNN
 F 1 "RFM69CW" H 9175 2925 60  0000 C CNN
-F 2 "" H 9225 2375 60  0000 C CNN
+F 2 "Hope_RFM:RFM69CW" H 9225 2375 60  0001 C CNN
 F 3 "" H 9225 2375 60  0000 C CNN
 	1    9225 2375
@@
 	8125 2075 8575 2075
 $Comp
-L GND #PWR?
+L GND #PWR021
 U 1 1 5805BB01
 P 8475 2675
-F 0 "#PWR?" H 8475 2425 50  0001 C CNN
+F 0 "#PWR021" H 8475 2425 50  0001 C CNN
 F 1 "GND" H 8475 2525 50  0000 C CNN
 F 2 "" H 8475 2675 50  0000 C CNN
@@
 	9900 2375 9900 2725
 $Comp
-L GND #PWR?
+L GND #PWR022
 U 1 1 5805C11A
 P 9900 2725
-F 0 "#PWR?" H 9900 2475 50  0001 C CNN
+F 0 "#PWR022" H 9900 2475 50  0001 C CNN
 F 1 "GND" H 9900 2575 50  0000 C CNN
 F 2 "" H 9900 2725 50  0000 C CNN
@@
 	9950 2475 9950 1700
 $Comp
-L VDD #PWR?
+L VDD #PWR023
 U 1 1 5805C214
 P 9950 1700
-F 0 "#PWR?" H 9950 1550 50  0001 C CNN
+F 0 "#PWR023" H 9950 1550 50  0001 C CNN
 F 1 "VDD" H 9950 1850 50  0000 C CNN
 F 2 "" H 9950 1700 50  0000 C CNN
@@
 	9825 2575 10475 2575
 $Comp
-L CONN_01X01 P?
+L CONN_01X01 P2003
 U 1 1 5805C2C3
 P 10600 2575
-F 0 "P?" H 10600 2675 50  0000 C CNN
+F 0 "P2003" H 10600 2675 50  0000 C CNN
 F 1 "antenna" V 10700 2575 50  0000 C CNN
-F 2 "" H 10600 2575 50  0000 C CNN
+F 2 "Socket_Strips:Socket_Strip_Straight_1x01" H 10600 2575 50  0001 C CNN
 F 3 "" H 10600 2575 50  0000 C CNN
 	1    10600 2575
@@
 $EndComp
 $Comp
-L CONN_02X04 P?
+L CONN_02X04 P2001
 U 1 1 5805CADD
 P 5050 5100
-F 0 "P?" H 5050 5350 50  0000 C CNN
-F 1 "CONN_02X04" H 5050 4850 50  0000 C CNN
-F 2 "" H 5050 3900 50  0000 C CNN
+F 0 "P2001" H 5050 5350 50  0000 C CNN
+F 1 "WIFI" H 5050 4850 50  0000 C CNN
+F 2 "Socket_Strips:Socket_Strip_Straight_2x04" H 5050 3900 50  0001 C CNN
 F 3 "" H 5050 3900 50  0000 C CNN
 	1    5050 5100
@@
 $EndComp
 $Comp
-L CONN_01X07 P?
+L CONN_01X07 P2002
 U 1 1 5805CC77
 P 5100 6300
-F 0 "P?" H 5100 6700 50  0000 C CNN
-F 1 "CONN_01X07" V 5200 6300 50  0000 C CNN
-F 2 "" H 5100 6300 50  0000 C CNN
+F 0 "P2002" H 5100 6700 50  0000 C CNN
+F 1 "GPRS" V 5200 6300 50  0000 C CNN
+F 2 "Socket_Strips:Socket_Strip_Straight_1x07" H 5100 6300 50  0001 C CNN
 F 3 "" H 5100 6300 50  0000 C CNN
 	1    5100 6300
 	1    0    0    -1
 $EndComp
-Text Notes 5425 4650 2    60   ~ 0
-ESP-01 connector
-Text Notes 5425 5825 2    60   ~ 0
-M590E connector
+Text Notes 5775 4775 2    60   ~ 0
+ESP-01 or ESP-12 connector
+Text Notes 5600 5825 2    60   ~ 0
+M590E or A6 connector
+Text HLabel 1625 3200 0    60   Input ~ 0
+data_rx
+Wire Wire Line
+	1625 3200 2125 3200
+Text HLabel 1625 3575 0    60   Output ~ 0
+data_tx
+Wire Wire Line
+	1625 3575 2125 3575
+Text HLabel 1600 4225 0    60   Input ~ 0
+data_enable
+Text HLabel 1625 4575 0    60   Input ~ 0
+data_reset
+Text HLabel 1325 950  0    60   Input ~ 0
+RF_CS
+Text HLabel 1500 4825 0    60   Input ~ 0
+data_io0
+Text HLabel 1575 4950 0    60   Input ~ 0
+data_io1
 $EndSCHEMATC
