File: Hardware/digital/kicad/digital-a.kicad_pcb (KiCad board)
At the start: 2 copper layers, 135 x 95 mm, 40 parts, among them IC101 ATMEGA1284-P, P101 Power, P102 Analog, P103 PWM, P104 PWM, P105 Communication, P106 h2, P107 h3, P108 h4, P109 h5, P110 h6, P111 h7, P112 h8, P113 5VDC, P114 POWER_SOURCE, P115 CONN_01X04, P116 CONN_01X04, P201 SD CARD, SW101 Switch_DPST, X601 10M, X602 CRYSTAL

Commit message: update digital files
Parts:
- removed C101: 1u, Capacitors_ThroughHole:C_Radial_D5_L6_P2.5
- removed C201, C202, C203, C204: 47p, Capacitors_ThroughHole:C_Rect_L7_W2.5_P5
- removed C601, C603, C604, C607, C608: 100n, Capacitors_ThroughHole:C_Rect_L7_W2.5_P5
- removed C605, C606, C609, C610: 20p, Capacitors_ThroughHole:C_Rect_L7_W2.5_P5
- removed IC101: ATMEGA1284-P, Housings_DIP:DIP-40_W15.24mm_LongPads
- removed R201, R202, R203: 100k, Resistors_ThroughHole:Resistor_Horizontal_RM10mm
- removed R601: 330, Resistors_ThroughHole:Resistor_Horizontal_RM10mm
- removed R602: 10k, Resistors_ThroughHole:Resistor_Horizontal_RM10mm
- removed SW101: Switch_DPST, Buttons_Switches_ThroughHole:SW_TH_Tactile_Omron_B3F-10xx
- removed X601: 10M, Crystals:Crystal_HC50-U_Vertical
- removed X602: CRYSTAL, Crystals:Crystal_Round_Horizontal_3mm_BigPad
- added P2001: WIFI, Socket_Strips:Socket_Strip_Straight_2x04, F.Cu at (165.6, 100.8)
- added P2002: GPRS, Socket_Strips:Socket_Strip_Straight_1x07, F.Cu at (160.0, 108.2)
- added U2002: RFM69CW, Hope_RFM:RFM69CW, F.Cu at (193.9, 125.2)
- moved P201 72.7 mm to (164.7, 130.3)
Connections:
- P101 pad 1: (no net) -> Net-(P101-Pad1)
- P101 pad 2: (no net) -> Net-(P101-Pad2)
- P101 pad 4: (no net) -> Net-(P101-Pad4)
- P101 pad 5: (no net) -> Net-(P101-Pad5)
- P101 pad 8: (no net) -> Net-(P101-Pad8)
- P103 pad 10: (no net) -> /sd_cs1
- P103 pad 9: (no net) -> /sd_cs2
- P106 pad 1: (no net) -> Net-(P106-Pad1)
- P107 pad 1: (no net) -> Net-(P107-Pad1)
- P108 pad 1: (no net) -> Net-(P108-Pad1)
- P109 pad 1: (no net) -> Net-(P109-Pad1)
- P110 pad 1: (no net) -> Net-(P110-Pad1)
- P111 pad 1: (no net) -> Net-(P111-Pad1)
- P112 pad 1: (no net) -> Net-(P112-Pad1)
- P201 pad 2: (no net) -> Net-(P201-Pad2)
- P201 pad 4: (no net) -> Net-(P201-Pad4)
- P201 pad 6: (no net) -> Net-(P201-Pad6)
- P201 pad 7: (no net) -> VAA
Other:
- board text added: "GPRS"
- board text added: "SD card"
- board text added: "SPI modules"
- board text added: "UART modules"
- board text added: "WIFI"
