File: Hardware/digital/kicad/digital-a.sch (KiCad schematic (older format))
At the start: 32 parts, among them IC101 ATMEGA1284-P, P101 Power, P102 Analog, P103 PWM, P104 PWM, P105 Communication, P106 h2, P107 h3, P108 h4, P109 h5, P110 h6, P111 h7, P112 h8, P113 5VDC, P114 POWER_SOURCE, P115 CONN_01X04, P116 CONN_01X04, SW101 Switch_DPST, X601 10M, X602 CRYSTAL

Commit message: update digital files
Connections:
- net labels added: RF_CS, data_enable
- net labels removed: SD1_power, SD2_power, data_power
- wire segments 138 -> 145
Other:
- note added: "- SD card connector\n- transmitter's connector\nfor wifi or gprs"
- note added: "Arduino style but with Atmega 1284P"
- note added: "Main crystal"
- note added: "RTC crystal"
- note added: "Reset button"
- note added: "ftdi USB/USART converter\nfor the PC communication\n and a ISP connector"
- note added: "mecanic holes"
- note removed: "Main oscillator"
- moved on the sheet: C101, C601, C603, C604, C605, C606, C607, C608, C609, C610, IC101, P101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
