File: Hardware/digital/kicad/digital.kicad_pcb (KiCad board)
At the start: 2 copper layers, 120 x 128 mm, 93 parts, among them IC1 ATMEGA1284P-A, J1 CONN-SMA-5-1814400-1, J2 Micro_SD, P1 CONN_01X14, P11 USB_OTG, P12 CONN_01X02, P13 CONN_01X02, P2 CONN_01X14, P3 ISP, P4 CONN_02X05, P5 hole, P6 hole, P7 USART0, P8 hole, P9 hole, Q1 NTR4501N, Q2 FQB22P10, Q3 FQB22P10, SW1 button-touch-6x6mm, SW2 button-touch-6x6mm, U1 FT232RL, U2 EPM3064A-44TQFP, U3 RFM69CW, U4 SIM800L, U5 huzzah, U6 LM3485, U7 LM1085IS-3.3/NOPB, U8 LM358, X1 16M, X2 CRYSTAL, X3 32MHz

Commit message: move to digital v1.0.1
Parts:
- added D12: Led_Small, LEDs:LED-3MM, F.Cu at (86.3, 85.5)
- added R13: 270, Discret:R3-LARGE_PADS, F.Cu at (85.7, 74.8)
- R8: value 100 -> 270
Routing:
- net /CPLD/10: track 90.6 -> 113.2 mm
- net Net-(D12-Pad2): track 0.00 -> 4.53 mm
- net GND: track 1223.2 -> 1223.7 mm, vias 28 -> 27
Other:
- board text added: "Windlogger project digital board v1.0.1"
- board text removed: "Windlogger project digital board v1.0.0"
Changed lines of the file:
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@@
 (kicad_pcb (version 4) (host pcbnew 4.0.2+dfsg1-2~bpo8+1-stable)
   (general
-    (links 317)
+    (links 320)
     (no_connects 0)
     (area 76.108 32.411 202.042524 164.231)
     (thickness 1.6)
     (drawings 63)
-    (tracks 2371)
+    (tracks 2384)
     (zones 0)
-    (modules 93)
-    (nets 92)
+    (modules 95)
+    (nets 93)
   )
   (page A4)
+  (title_block
+    (title "Windlogger digital")
+    (date 2017-02-02)
+    (rev 1.0.1)
+    (company ALEEA)
+    (comment 1 "LONGUET Gilles")
+    (comment 2 AGPL3)
+  )
   (layers
     (0 F.Cu signal)
@@
     (visible_elements FFFEFF7F)
     (pcbplotparams
-      (layerselection 0x00000_80000001)
+      (layerselection 0x01000_00000000)
       (usegerberextensions true)
       (excludeedgelayer true)
@@
   (net 90 "Net-(U8-Pad1)")
   (net 91 "Net-(Q2-Pad1)")
+  (net 92 "Net-(D12-Pad2)")
   (net_class Default "This is the default net class."
     (clearance 0.25)
@@
     (add_net /uart0_interace/CTS)
     (add_net /uart0_interace/DTR)
-    (add_net GND)
     (add_net "Net-(C13-Pad2)")
     (add_net "Net-(C14-Pad2)")
@@
     (add_net "Net-(D1-Pad2)")
     (add_net "Net-(D10-Pad1)")
+    (add_net "Net-(D12-Pad2)")
     (add_net "Net-(D2-Pad1)")
     (add_net "Net-(D2-Pad2)")
@@
     (uvia_dia 0.8)
     (uvia_drill 0.4)
+    (add_net GND)
   )
   (module Capacitors_ThroughHole:C_Rect_L4_W2.5_P2.5 (layer F.Cu)
@@
       (effects (font (size 1 1) (thickness 0.15)))
     )
-    (fp_text value 100 (at 0 0) (layer F.Fab)
+    (fp_text value 270 (at 0 0) (layer F.Fab)
       (effects (font (size 1 1) (thickness 0.15)))
     )
@@
       (net 23 /power_supply/FB_buck))
   )
+  (module LEDs:LED-3MM (layer F.Cu)
+    (at 86.252 85.482 90)
+    (descr "LED 3mm round vertical")
+    (tags "LED  3mm round vertical")
+    (fp_text reference D12 (at 1.91 3.06 90) (layer F.SilkS)
+      (effects (font (size 1 1) (thickness 0.15)))
+    )
+    (fp_text value Led_Small (at 1.3 -2.9 90) (layer F.Fab)
+      (effects (font (size 1 1) (thickness 0.15)))
+    )
+    (fp_line (start -1.2 2.3) (end 3.8 2.3) (layer F.CrtYd) (width 0.05))
+    (fp_line (start 3.8 2.3) (end 3.8 -2.2) (layer F.CrtYd) (width 0.05))
+    (fp_line (start 3.8 -2.2) (end -1.2 -2.2) (layer F.CrtYd) (width 0.05))
+    (fp_line (start -1.2 -2.2) (end -1.2 2.3) (layer F.CrtYd) (width 0.05))
+    (fp_line (start -0.199 1.314) (end -0.199 1.114) (layer F.SilkS) (width 0.15))
+    (fp_line (start -0.199 -1.28) (end -0.199 -1.1) (layer F.SilkS) (width 0.15))
+    (fp_arc (start 1.301 0.034) (end -0.199 -1.286) (angle 108.5) (layer F.SilkS) (width 0.15))
+    (fp_arc (start 1.301 0.034) (end 0.25 -1.1) (angle 85.7) (layer F.SilkS) (width 0.15))
+    (fp_arc (start 1.311 0.034) (end 3.051 0.994) (angle 110) (layer F.SilkS) (width 0.15))
+    (fp_arc (start 1.301 0.034) (end 2.335 1.094) (angle 87.5) (layer F.SilkS) (width 0.15))
+    (fp_text user K (at -1.69 1.74 90) (layer F.SilkS)
+      (effects (font (size 1 1) (thickness 0.15)))
+    )
+    (pad 1 thru_hole rect (at 0 0 180) (size 2 2) (drill 1.00076) (layers *.Cu *.Mask F.SilkS)
+      (net 10 GND))
+    (pad 2 thru_hole circle (at 2.54 0 90) (size 2 2) (drill 1.00076) (layers *.Cu *.Mask F.SilkS)
+      (net 92 "Net-(D12-Pad2)"))
+    (model LEDs.3dshapes/LED-3MM.wrl
+      (at (xyz 0.05 0 0))
+      (scale (xyz 1 1 1))
+      (rotate (xyz 0 0 90))
+    )
+  )
+  (module Discret:R3-LARGE_PADS (layer F.Cu)
+    (at 85.744 74.814 90)
+    (descr "Resitance 3 pas")
+    (tags R)
+    (fp_text reference R13 (at 0 0 90) (layer F.SilkS)
+      (effects (font (size 1 1) (thickness 0.15)))
+    )
+    (fp_text value 270 (at 0 0 90) (layer F.Fab)
+      (effects (font (size 1 1) (thickness 0.15)))
+    )
+    (fp_line (start -3.81 0) (end -3.302 0) (layer F.SilkS) (width 0.15))
+    (fp_line (start 3.81 0) (end 3.302 0) (layer F.SilkS) (width 0.15))
+    (fp_line (start 3.302 0) (end 3.302 -1.016) (layer F.SilkS) (width 0.15))
+    (fp_line (start 3.302 -1.016) (end -3.302 -1.016) (layer F.SilkS) (width 0.15))
+    (fp_line (start -3.302 -1.016) (end -3.302 1.016) (layer F.SilkS) (width 0.15))
+    (fp_line (start -3.302 1.016) (end 3.302 1.016) (layer F.SilkS) (width 0.15))
+    (fp_line (start 3.302 1.016) (end 3.302 0) (layer F.SilkS) (width 0.15))
+    (fp_line (start -3.302 -0.508) (end -2.794 -1.016) (layer F.SilkS) (width 0.15))
+    (pad 1 thru_hole circle (at -3.81 0 90) (size 1.651 1.651) (drill 0.8128) (layers *.Cu *.Mask F.SilkS)
+      (net 92 "Net-(D12-Pad2)"))
+    (pad 2 thru_hole circle (at 3.81 0 90) (size 1.651 1.651) (drill 0.8128) (layers *.Cu *.Mask F.SilkS)
+      (net 47 /CPLD/10))
+    (model Discret.3dshapes/R3-LARGE_PADS.wrl
+      (at (xyz 0 0 0))
+      (scale (xyz 0.3 0.3 0.3))
+      (rotate (xyz 0 0 0))
+    )
+  )
   (gr_text "aleea.org\ntripalium.org" (at 142.378 141.666) (layer F.SilkS)
     (effects (font (size 2 2) (thickness 0.3)))
   )
-  (gr_text "Windlogger project\ndigital board v1.0.0" (at 153.378 149.666) (layer F.SilkS)
+  (gr_text "Windlogger project\ndigital board v1.0.1" (at 153.378 149.666) (layer F.SilkS)
     (effects (font (size 3 3) (thickness 0.5)))
   )
@@
   (segment (start 114.738 104.316) (end 114.7 104.278) (width 0.25) (layer F.Cu) (net 9) (status 30))
   (segment (start 120.288 113.168) (end 120.288 112.613) (width 0.25) (layer F.Cu) (net 9) (status 30))
+  (via (at 80.156 85.482) (size 0.8) (drill 0.4) (layers F.Cu B.Cu) (net 10))
+  (segment (start 80.156 85.482) (end 80.283 85.482) (width 0.5) (layer F.Cu) (net 10))
+  (segment (start 80.156 85.482) (end 80.283 85.482) (width 0.5) (layer F.Cu) (net 10))
+  (segment (start 86.252 85.482) (end 80.156 85.482) (width 0.5) (layer B.Cu) (net 10))
+  (segment (start 90.57 85.736) (end 86.506 85.736) (width 0.5) (layer F.Cu) (net 10))
+  (segment (start 86.506 85.736) (end 86.252 85.482) (width 0.5) (layer F.Cu) (net 10))
   (segment (start 185.098 89.546) (end 185.098 90.094) (width 0.25) (layer F.Cu) (net 10))
   (segment (start 185.098 90.094) (end 186.328 91.324) (width 0.25) (layer F.Cu) (net 10))
@@
   (segment (start 111.398 85.101) (end 110.763 85.736) (width 0.25) (layer B.Cu) (net 10))
   (segment (start 86.558 99.416) (end 86.558 94.916) (width 0.25) (layer B.Cu) (net 10) (status 30))
-  (via (at 80.283 85.736) (size 0.8) (drill 0.4) (layers F.Cu B.Cu) (net 10))
   (via (at 110.763 85.736) (size 0.8) (drill 0.4) (layers F.Cu B.Cu) (net 10))
-  (segment (start 110.763 85.736) (end 84.728 85.736) (width 0.5) (layer F.Cu) (net 10))
-  (via (at 84.728 85.736) (size 0.8) (drill 0.4) (layers F.Cu B.Cu) (net 10))
-  (segment (start 84.728 85.736) (end 80.283 85.736) (width 0.5) (layer B.Cu) (net 10))
+  (segment (start 110.763 85.736) (end 90.57 85.736) (width 0.5) (layer F.Cu) (net 10))
   (segment (start 119.018 122.126) (end 119.018 119.518) (width 0.25) (layer B.Cu) (net 10) (status 10))
   (segment (start 119.018 119.518) (end 120.288 118.168) (width 0.25) (layer B.Cu) (net 10) (status 20))
@@
   (segment (start 98.698 64.146) (end 96.793 66.051) (width 1) (layer F.Cu) (net 10))
   (segment (start 103.778 64.146) (end 98.698 64.146) (width 1) (layer F.Cu) (net 10))
-  (segment (start 80.283 66.686) (end 80.283 85.736) (width 1) (layer F.Cu) (net 10))
+  (segment (start 80.283 66.686) (end 80.283 85.482) (width 1) (layer F.Cu) (net 10))
+  (segment (start 80.283 85.482) (end 80.283 85.736) (width 1) (layer F.Cu) (net 10))
   (segment (start 80.918 66.051) (end 80.283 66.686) (width 1) (layer F.Cu) (net 10))
   (segment (start 96.793 66.051) (end 80.918 66.051) (width 1) (layer F.Cu) (net 10))
@@
   (segment (start 144.926 104.278) (end 141.878 104.278) (width 0.25) (layer F.Cu) (net 46))
   (segment (start 145.684 105.036) (end 144.926 104.278) (width 0.25) (layer F.Cu) (net 46))
+  (segment (start 107.334 69.226) (end 103.524 69.226) (width 0.25) (layer F.Cu) (net 47))
+  (segment (start 92.602 71.004) (end 85.744 71.004) (width 0.25) (layer F.Cu) (net 47))
+  (segment (start 94.179994 69.426006) (end 92.602 71.004) (width 0.25) (layer F.Cu) (net 47))
+  (segment (start 95.596006 69.426006) (end 94.179994 69.426006) (width 0.25) (layer F.Cu) (net 47))
+  (segment (start 95.904 69.734) (end 95.596006 69.426006) (width 0.25) (layer F.Cu) (net 47))
+  (segment (start 103.016 69.734) (end 95.904 69.734) (width 0.25) (layer F.Cu) (net 47))
+  (segment (start 103.524 69.226) (end 103.016 69.734) (width 0.25) (layer F.Cu) (net 47))
   (segment (start 129.178 91.07) (end 127.4 91.07) (width 0.25) (layer F.Cu) (net 47))
   (segment (start 131.718 93.61) (end 129.178 91.07) (width 0.25) (layer F.Cu) (net 47) (status 10))
@@
   (via (at 108.223 50.811) (size 0.8) (drill 0.4) (layers F.Cu B.Cu) (net 91))
   (segment (start 112.033 50.811) (end 108.223 50.811) (width 0.25) (layer B.Cu) (net 91))
+  (segment (start 86.252 82.942) (end 86.252 79.132) (width 0.25) (layer B.Cu) (net 92))
+  (segment (start 86.252 79.132) (end 85.744 78.624) (width 0.25) (layer B.Cu) (net 92))
   (zone (net 82) (net_name "Net-(P11-Pad6)") (layer B.Cu) (hatch edge 0.508)
     (connect_pads (clearance 0.3))
