File: Hardware/digital/kicad/uart0_interace.sch (KiCad schematic (older format))
At the start: 11 parts, among them P11 USB_OTG, U1 FT232RL

Commit message: move to digital v1.0.1
Parts:
- R1, R2: value 1k -> 270
Changed lines of the file:
@@
 EESchema Schematic File Version 2
 LIBS:ftdi
-LIBS:digital-a-rescue
 LIBS:power
 LIBS:device
@@
 LIBS:Hope_RFM
 LIBS:digital
-LIBS:altera
 LIBS:Oscillators
-LIBS:IHE
-LIBS:conn-te
 LIBS:dc-dc
 LIBS:digital-cache
@@
 Sheet 2 6
 Title "Windlogger digital"
-Date "2017-01-24"
-Rev "1.0.0"
+Date "2017-02-02"
+Rev "1.0.1"
 Comp "ALEEA"
 Comment1 "LONGUET Gilles"
@@
 $EndComp
 $Comp
-L GND #PWR09
+L GND #PWR010
 U 1 1 586F20A9
 P 3275 4550
-F 0 "#PWR09" H 3275 4300 50  0001 C CNN
+F 0 "#PWR010" H 3275 4300 50  0001 C CNN
 F 1 "GND" H 3275 4400 50  0000 C CNN
 F 2 "" H 3275 4550 50  0000 C CNN
@@
 	3475 2950 3475 3825
 $Comp
-L GND #PWR010
+L GND #PWR011
 U 1 1 586F27D9
 P 3825 4300
-F 0 "#PWR010" H 3825 4050 50  0001 C CNN
+F 0 "#PWR011" H 3825 4050 50  0001 C CNN
 F 1 "GND" H 3825 4150 50  0000 C CNN
 F 2 "" H 3825 4300 50  0000 C CNN
@@
 $EndComp
 $Comp
-L +3.3V #PWR011
+L +3.3V #PWR012
 U 1 1 586F2898
 P 4125 3200
-F 0 "#PWR011" H 4125 3050 50  0001 C CNN
+F 0 "#PWR012" H 4125 3050 50  0001 C CNN
 F 1 "+3.3V" H 4125 3340 50  0000 C CNN
 F 2 "" H 4125 3200 50  0000 C CNN
@@
 Connection ~ 4125 3225
 $Comp
-L +5V #PWR012
+L +5V #PWR013
 U 1 1 586F2BB2
 P 5850 2800
-F 0 "#PWR012" H 5850 2650 50  0001 C CNN
+F 0 "#PWR013" H 5850 2650 50  0001 C CNN
 F 1 "+5V" H 5850 2940 50  0000 C CNN
 F 2 "" H 5850 2800 50  0000 C CNN
@@
 	5850 2800 5850 2925
 $Comp
-L GND #PWR013
+L GND #PWR014
 U 1 1 586F2F97
 P 4700 4750
-F 0 "#PWR013" H 4700 4500 50  0001 C CNN
+F 0 "#PWR014" H 4700 4500 50  0001 C CNN
 F 1 "GND" H 4700 4600 50  0000 C CNN
 F 2 "" H 4700 4750 50  0000 C CNN
@@
 $EndComp
 $Comp
-L GND #PWR014
+L GND #PWR015
 U 1 1 586F2FB7
 P 5750 5050
-F 0 "#PWR014" H 5750 4800 50  0001 C CNN
+F 0 "#PWR015" H 5750 4800 50  0001 C CNN
 F 1 "GND" H 5750 4900 50  0000 C CNN
 F 2 "" H 5750 5050 50  0000 C CNN
@@
 P 7325 3675
 F 0 "R1" V 7405 3675 50  0000 C CNN
-F 1 "1k" V 7325 3675 50  0000 C CNN
+F 1 "270" V 7325 3675 50  0000 C CNN
 F 2 "Discret:R3-LARGE_PADS" V 7255 3675 50  0001 C CNN
 F 3 "" H 7325 3675 50  0000 C CNN
@@
 P 7725 3675
 F 0 "R2" V 7805 3675 50  0000 C CNN
-F 1 "1k" V 7725 3675 50  0000 C CNN
+F 1 "270" V 7725 3675 50  0000 C CNN
 F 2 "Discret:R3-LARGE_PADS" V 7655 3675 50  0001 C CNN
 F 3 "" H 7725 3675 50  0000 C CNN
@@
 	7725 3425 7725 3525
 $Comp
-L +5V #PWR015
+L +5V #PWR016
 U 1 1 586F3EB6
 P 7525 3375
-F 0 "#PWR015" H 7525 3225 50  0001 C CNN
+F 0 "#PWR016" H 7525 3225 50  0001 C CNN
 F 1 "+5V" H 7525 3515 50  0000 C CNN
 F 2 "" H 7525 3375 50  0000 C CNN
@@
 	8300 3925 8300 3875
 $Comp
-L +5V #PWR016
+L +5V #PWR017
 U 1 1 586FAB39
 P 8300 3875
-F 0 "#PWR016" H 8300 3725 50  0001 C CNN
+F 0 "#PWR017" H 8300 3725 50  0001 C CNN
 F 1 "+5V" H 8300 4015 50  0000 C CNN
 F 2 "" H 8300 3875 50  0000 C CNN
