File: Hardware/digital/kicad/digital.sch (KiCad schematic (older format))
At the start: 16 parts, among them P1 CONN_01X14, P2 CONN_01X14, P3 ISP, P4 CONN_02X05, P5 hole, P6 hole, P7 USART0, P8 hole, P9 hole

Commit message: move to digital v1.0.1
Parts:
- added D12: Led_Small, LEDs:LED-3MM, symbol Led_Small
- added R13: 270, Discret:R3-LARGE_PADS, symbol R
Connections:
- net D13-SCLK: now also R13.2
- net GND: now also D12.1 (K)
- new net: D12.2 (A), R13.1
Changed lines of the file:
@@
 EESchema Schematic File Version 2
 LIBS:ftdi
-LIBS:digital-a-rescue
 LIBS:power
 LIBS:device
@@
 LIBS:Hope_RFM
 LIBS:digital
-LIBS:altera
 LIBS:Oscillators
-LIBS:IHE
-LIBS:conn-te
 LIBS:dc-dc
 LIBS:digital-cache
@@
 Sheet 1 6
 Title "Windlogger digital"
-Date "2017-01-24"
-Rev "1.0.0"
+Date "2017-02-02"
+Rev "1.0.1"
 Comp "ALEEA"
 Comment1 "LONGUET Gilles"
@@
 Wire Wire Line
 	11000 1350 11000 1375
+Text Label 4875 1350 2    60   ~ 0
+D13-SCLK
+$Comp
+L R R13
+U 1 1 5892FF65
+P 5125 1350
+F 0 "R13" V 5205 1350 50  0000 C CNN
+F 1 "270" V 5125 1350 50  0000 C CNN
+F 2 "Discret:R3-LARGE_PADS" V 5055 1350 50  0001 C CNN
+F 3 "" H 5125 1350 50  0000 C CNN
+	1    5125 1350
+	0    1    1    0
+$EndComp
+$Comp
+L Led_Small D12
+U 1 1 58930F4F
+P 5500 1350
+F 0 "D12" H 5450 1475 50  0000 L CNN
+F 1 "Led_Small" H 5325 1250 50  0000 L CNN
+F 2 "LEDs:LED-3MM" V 5500 1350 50  0001 C CNN
+F 3 "" V 5500 1350 50  0000 C CNN
+	1    5500 1350
+	-1   0    0    1
+$EndComp
+$Comp
+L GND #PWR09
+U 1 1 589311BC
+P 5725 1350
+F 0 "#PWR09" H 5725 1100 50  0001 C CNN
+F 1 "GND" H 5725 1200 50  0000 C CNN
+F 2 "" H 5725 1350 50  0000 C CNN
+F 3 "" H 5725 1350 50  0000 C CNN
+	1    5725 1350
+	1    0    0    -1
+$EndComp
+Wire Wire Line
+	5725 1350 5600 1350
+Wire Wire Line
+	5400 1350 5275 1350
+Wire Wire Line
+	4975 1350 4875 1350
 $EndSCHEMATC

Commit message: move to digital 1.1.1
Parts:
- removed P1, P2: CONN_01X14, Socket_Strips:Socket_Strip_Straight_1x14, symbol CONN_01X14
- removed P4: CONN_02X05, Pin_Headers:Pin_Header_Straight_2x05, symbol CONN_02X05
- Analog1, PWM2, Power1: footprint Socket_Strips:Socket_Strip_Straight_1x08 -> digital:Socket_Strip_Straight_1x08
- C1: renamed from C2; value 100nF -> 100n
- P1: renamed from P7; footprint Pin_Headers:Pin_Header_Straight_1x06 -> digital:uart_usb_cp2102_module
- P3: footprint Socket_Strips:Socket_Strip_Straight_2x03 -> digital:Socket_Strip_Straight_2x03
- P5, P6, P8, P9: footprint Socket_Arduino_Mega:Arduino_1pin -> Mounting_Holes:MountingHole_3-5mm
- POWER_SOURCE1: footprint Socket_Strips:Socket_Strip_Straight_1x04 -> digital:Socket_Strip_Straight_1x04
- PWM1: footprint Socket_Strips:Socket_Strip_Straight_1x10 -> digital:Socket_Strip_Straight_1x10
- R1: renamed from R13; footprint Discret:R3-LARGE_PADS -> Resistors_ThroughHole:Resistor_Horizontal_RM10mm
- renumbered D12 to D1
Connections:
- net uart0_interace/CTS is gone; now on net GND: P1.2 (P2)
- net +5V: no longer P1.3 (P3)
- net DTR: now also P1.5 (P5); no longer P1.6 (P6)
- net GND: no longer P1.1 (P1)
- net D0-RX0 renamed D0_RX0+
- net D0_RX0+: now also P1.3 (P3); no longer P1.4 (P4)
- net D1-TX0 renamed D1_TX0-
- net D1_TX0-: now also P1.4 (P4); no longer P1.5 (P5)
- net power_supply/GND renamed power_supply/GND_PWR
- new net USBVCC: P1.1 (P1)
- no-connect marks 9 -> 7
Other:
- note added: "+5V\nGND\nTX0\nRX0\nDTR\n3V3"
- note added: "3.3V not connected"
- note added: "Microcontroler Uart to USB bridge"
- note removed: "+5V"
- note removed: "CPLD Jtag connector"
- note removed: "CTS"
- note removed: "DTR"
- note removed: "GND"
- note removed: "Microcontroler Uart"
- note removed: "RXI"
- note removed: "TXO"
- moved on the sheet: C1, D1, P1, POWER_SOURCE1, R1
