File: Hardware/digital/kicad/microC.sch (KiCad schematic (older format))
At the start: 14 parts, among them IC1 ATMEGA1284P-A, SW1 button-touch-6x6mm, X1 16M, X2 CRYSTAL

Commit message: move to digital 1.1.1
Parts:
- removed C12, C6: 100nF, Capacitors_ThroughHole:C_Rect_L7_W2.5_P5, symbol C
- removed IC1: ATMEGA1284P-A, Housings_QFP:TQFP-44_10x10mm_Pitch0.8mm, symbol ATMEGA1284P-A
- added IC1: ATMEGA1284P-P, Housings_DIP:DIP-40_W15.24mm_LongPads, symbol ATMEGA1284P-P
- C4: renamed from C9; value 100nF -> 100n
- C5: renamed from C10; value 100nF -> 100n
- C6: renamed from C11; value 100nF -> 100n
- C7: renamed from C13; value 12.5p -> 12p
- C8: renamed from C14; value 12.5p -> 12p
- R2: renamed from R4; value 10k -> 470k; footprint Discret:R3-LARGE_PADS -> Resistors_ThroughHole:Resistor_Horizontal_RM10mm
- X2: value CRYSTAL -> 32.768Hz
- renumbered C7 to C2, C8 to C3
Connections:
- net +5V: now also IC1.10 (VCC), IC1.30 (AVCC)
- net ACD0: now also IC1.40 ((PCINT0/ADC0)PA0)
- net ACD1: now also IC1.39 ((PCINT1/ADC1)PA1)
- net ACD2: now also IC1.38 ((PCINT2/ADC2)PA2)
- net ACD3: now also IC1.37 ((PCINT3/ADC3)PA3)
- net ACD4: now also IC1.36 ((PCINT4/ADC4)PA4)
- net ACD5: now also IC1.35 ((PCINT5/ADC5)PA5)
- net ACD6: now also IC1.34 ((PCINT6/ADC6)PA6)
- net ACD7: now also IC1.33 ((PCINT7/ADC7)PA7)
- net AREF: now also IC1.32 (AREF)
- net GND: now also IC1.11 (GND), IC1.31 (GND)
- net PB0: now also IC1.1 ((PCINT8/T0/XCK)PB0)
- net PB1: now also IC1.2 ((PCINT9/CLKO/T1)PB1)
- net PB2: now also IC1.3 ((PCINT10/AIN0/INT2)PB2)
- net PB3: now also IC1.4 ((PCINT11/AIN1/OC0)PB3)
- net PB4: now also IC1.5 ((PCINT12/OC0B/~SS~)PB4)
- net PB5: now also IC1.6 ((PCINT13/MOSI)PB5)
- net PB6: now also IC1.7 ((PCINT14/MISO)PB6)
- net PB7: now also IC1.8 ((PCINT15/SCK)PB7)
- net PC0: now also IC1.22 ((PCINT16/SCL)PC0)
- net PC1: now also IC1.23 ((PCINT17/SDA)PC1)
- net PC2: now also IC1.24 ((PCINT18/TCK)PC2)
- net PC3: now also IC1.25 ((PCINT19/TMS)PC3)
- net PC4: now also IC1.26 ((PCINT20/TDO)PC4)
- net PC5: now also IC1.27 ((PCINT21/TDI)PC5)
- net PD0: now also IC1.14 ((PCINT24/RXD0)PD0)
- net PD1: now also IC1.15 ((PCINT25/TXD0)PD1)
- net PD2: now also IC1.16 ((PCINT26/RXD1/INT0)PD2)
- net PD3: now also IC1.17 ((PCINT27/TXD1/INT1)PD3)
- net PD4: now also IC1.18 ((PCINT28/XCK1/OC1B)PD4)
- net PD5: now also IC1.19 ((PCINT294/OC1A)PD5)
- net PD6: now also IC1.20 ((PCINT30/OC2B/ICP)PD6)
- net PD7: now also IC1.21 ((PCINT31/OC2A)PD7)
- net RESET: now also IC1.9 (~RESET)
- net at C2.2, X1.2: now also IC1.12 (XTAL2)
- net at C3.2, X1.1: now also IC1.13 (XTAL1)
- net at C8.2, X2.1: now also IC1.29 ((PCINT23/TOSC2)PC7)
- net at C7.2, X2.2: now also IC1.28 ((PCINT22/TOSC1)PC6)
Other:
- note added: "Vérifier si on peut trouver un quartz avec condensateur 6pF dans ce cas pas besoin de C externe"
- moved on the sheet: C5, C6
Changed lines of the file:
@@
 EESchema Schematic File Version 2
+LIBS:digital
 LIBS:ftdi
 LIBS:power
@@
 LIBS:valves
 LIBS:Hope_RFM
-LIBS:digital
 LIBS:Oscillators
 LIBS:dc-dc
+LIBS:lm2672
 LIBS:digital-cache
 EELAYER 25 0
@@
 $Descr A4 11693 8268
 encoding utf-8
-Sheet 3 6
+Sheet 2 4
 Title "Windlogger digital"
-Date "2017-02-02"
-Rev "1.0.1"
+Date "2017-03-28"
+Rev "1.1.1"
 Comp "ALEEA"
 Comment1 "LONGUET Gilles"
@@
 $EndDescr
 $Comp
-L C C7
+L C C2
 U 1 1 58752FE3
 P 3825 2575
-F 0 "C7" H 3825 2675 40  0000 L CNN
+F 0 "C2" H 3825 2675 40  0000 L CNN
 F 1 "18p" H 3831 2490 40  0000 L CNN
 F 2 "Capacitors_ThroughHole:C_Rect_L4_W2.5_P2.5" H 3925 2425 30  0001 C CNN
@@
 $EndComp
 $Comp
-L C C8
+L C C3
 U 1 1 58752FEA
 P 3825 2975
-F 0 "C8" H 3825 3075 40  0000 L CNN
+F 0 "C3" H 3825 3075 40  0000 L CNN
 F 1 "18p" H 3831 2890 40  0000 L CNN
 F 2 "Capacitors_ThroughHole:C_Rect_L4_W2.5_P2.5" H 3863 2825 30  0001 C CNN
@@
 $EndComp
 $Comp
-L C C6
-U 1 1 58752FF1
-P 5600 1775
-F 0 "C6" H 5600 1875 40  0000 L CNN
-F 1 "100nF" H 5606 1690 40  0000 L CNN
-F 2 "Capacitors_ThroughHole:C_Rect_L7_W2.5_P5" H 5700 1625 30  0001 C CNN
-F 3 "~" H 5600 1775 60  0000 C CNN
-	1    5600 1775
-	0    -1   -1   0
-$EndComp
-$Comp
-L R R4
+L R R2
 U 1 1 58752FF8
 P 3275 1950
-F 0 "R4" V 3355 1950 40  0000 C CNN
-F 1 "10k" V 3282 1951 40  0000 C CNN
-F 2 "Discret:R3-LARGE_PADS" V 3205 1950 30  0001 C CNN
+F 0 "R2" V 3355 1950 40  0000 C CNN
+F 1 "470k" V 3282 1951 40  0000 C CNN
+F 2 "Resistors_ThroughHole:Resistor_Horizontal_RM10mm" V 3205 1950 30  0001 C CNN
 F 3 "~" H 3275 1950 30  0000 C CNN
 	1    3275 1950
@@
 $EndComp
 $Comp
-L C C10
+L C C5
 U 1 1 58752FFF
-P 2900 3850
-F 0 "C10" H 2900 3950 40  0000 L CNN
-F 1 "100nF" H 2906 3765 40  0000 L CNN
-F 2 "Capacitors_ThroughHole:C_Rect_L7_W2.5_P5" H 3000 3700 30  0001 C CNN
-F 3 "~" H 2900 3850 60  0000 C CNN
-	1    2900 3850
-	1    0    0    -1
-$EndComp
-$Comp
-L C C11
+P 2400 5450
+F 0 "C5" H 2400 5550 40  0000 L CNN
+F 1 "100n" H 2406 5365 40  0000 L CNN
+F 2 "Capacitors_ThroughHole:C_Rect_L7_W2.5_P5" H 2500 5300 30  0001 C CNN
+F 3 "~" H 2400 5450 60  0000 C CNN
+	1    2400 5450
+	1    0    0    -1
+$EndComp
+$Comp
+L C C6
 U 1 1 58753006
-P 3200 3850
-F 0 "C11" H 3200 3950 40  0000 L CNN
-F 1 "100nF" H 3206 3765 40  0000 L CNN
-F 2 "Capacitors_ThroughHole:C_Rect_L7_W2.5_P5" H 3300 3700 30  0001 C CNN
-F 3 "~" H 3200 3850 60  0000 C CNN
-	1    3200 3850
-	1    0    0    -1
-$EndComp
-$Comp
-L C C12
-U 1 1 5875300D
-P 3500 3850
-F 0 "C12" H 3500 3950 40  0000 L CNN
-F 1 "100nF" H 3506 3765 40  0000 L CNN
-F 2 "Capacitors_ThroughHole:C_Rect_L7_W2.5_P5" H 3600 3700 30  0001 C CNN
-F 3 "~" H 3500 3850 60  0000 C CNN
-	1    3500 3850
+P 2700 5450
+F 0 "C6" H 2700 5550 40  0000 L CNN
+F 1 "100n" H 2706 5365 40  0000 L CNN
+F 2 "Capacitors_ThroughHole:C_Rect_L7_W2.5_P5" H 2800 5300 30  0001 C CNN
+F 3 "~" H 2700 5450 60  0000 C CNN
+	1    2700 5450
 	1    0    0    -1
 $EndComp
@@
 AREF
 $Comp
-L C C9
+L C C4
 U 1 1 5875301E
 P 3975 3600
-F 0 "C9" H 3975 3700 40  0000 L CNN
-F 1 "100nF" H 3981 3515 40  0000 L CNN
+F 0 "C4" H 3975 3700 40  0000 L CNN
+F 1 "100n" H 3981 3515 40  0000 L CNN
 F 2 "Capacitors_ThroughHole:C_Rect_L7_W2.5_P5" H 4075 3450 30  0001 C CNN
 F 3 "~" H 3975 3600 60  0000 C CNN
@@
 P 7225 4675
 F 0 "X2" V 7425 4625 60  0000 C CNN
-F 1 "CRYSTAL" V 7000 4650 60  0000 C CNN
+F 1 "32.768Hz" V 7000 4650 60  0000 C CNN
 F 2 "Crystals:Crystal_Round_Horizontal_3mm_BigPad" H 7225 4675 60  0001 C CNN
 F 3 "" H 7225 4675 60  0000 C CNN
@@
 $EndComp
 $Comp
-L C C13
+L C C7
 U 1 1 58753031
 P 7550 4525
-F 0 "C13" H 7550 4625 40  0000 L CNN
-F 1 "12.5p" H 7556 4440 40  0000 L CNN
+F 0 "C7" H 7550 4625 40  0000 L CNN
+F 1 "12p" H 7556 4440 40  0000 L CNN
 F 2 "Capacitors_ThroughHole:C_Rect_L4_W2.5_P2.5" H 7588 4375 30  0001 C CNN
 F 3 "" H 7550 4525 60  0000 C CNN
@@
 $EndComp
 $Comp
-L C C14
+L C C8
 U 1 1 58753038
 P 7550 4825
-F 0 "C14" H 7550 4925 40  0000 L CNN
-F 1 "12.5p" H 7556 4740 40  0000 L CNN
+F 0 "C8" H 7550 4925 40  0000 L CNN
+F 1 "12p" H 7556 4740 40  0000 L CNN
 F 2 "Capacitors_ThroughHole:C_Rect_L4_W2.5_P2.5" H 7588 4675 30  0001 C CNN
 F 3 "" H 7550 4825 60  0000 C CNN
@@
 $EndComp
 $Comp
-L GND #PWR018
+L GND #PWR08
 U 1 1 5875303F
 P 7825 4675
-F 0 "#PWR018" H 7825 4425 50  0001 C CNN
+F 0 "#PWR08" H 7825 4425 50  0001 C CNN
 F 1 "GND" H 7825 4525 50  0000 C CNN
 F 2 "" H 7825 4675 50  0000 C CNN
@@
 $EndComp
 $Comp
-L GND #PWR019
+L GND #PWR09
 U 1 1 58753045
-P 2900 4050
-F 0 "#PWR019" H 2900 3800 50  0001 C CNN
-F 1 "GND" H 2900 3900 50  0000 C CNN
-F 2 "" H 2900 4050 50  0000 C CNN
-F 3 "" H 2900 4050 50  0000 C CNN
-	1    2900 4050
-	1    0    0    -1
-$EndComp
-$Comp
-L +5V #PWR020
+P 2400 5675
+F 0 "#PWR09" H 2400 5425 50  0001 C CNN
+F 1 "GND" H 2400 5525 50  0000 C CNN
+F 2 "" H 2400 5675 50  0000 C CNN
+F 3 "" H 2400 5675 50  0000 C CNN
+	1    2400 5675
+	1    0    0    -1
+$EndComp
+$Comp
+L +5V #PWR010
 U 1 1 5875304B
-P 2900 3650
-F 0 "#PWR020" H 2900 3500 50  0001 C CNN
-F 1 "+5V" H 2900 3790 50  0000 C CNN
-F 2 "" H 2900 3650 50  0000 C CNN
-F 3 "" H 2900 3650 50  0000 C CNN
-	1    2900 3650
-	1    0    0    -1
-$EndComp
-$Comp
-L GND #PWR021
+P 2400 5225
+F 0 "#PWR010" H 2400 5075 50  0001 C CNN
+F 1 "+5V" H 2400 5365 50  0000 C CNN
+F 2 "" H 2400 5225 50  0000 C CNN
+F 3 "" H 2400 5225 50  0000 C CNN
+	1    2400 5225
+	1    0    0    -1
+$EndComp
+$Comp
+L GND #PWR011
 U 1 1 58753051
 P 5125 5950
-F 0 "#PWR021" H 5125 5700 50  0001 C CNN
+F 0 "#PWR011" H 5125 5700 50  0001 C CNN
 F 1 "GND" H 5125 5800 50  0000 C CNN
 F 2 "" H 5125 5950 50  0000 C CNN
@@
 $EndComp
 $Comp
-L GND #PWR022
+L GND #PWR012
 U 1 1 58753057
 P 3975 3800
-F 0 "#PWR022" H 3975 3550 50  0001 C CNN
+F 0 "#PWR012" H 3975 3550 50  0001 C CNN
 F 1 "GND" H 3975 3650 50  0000 C CNN
 F 2 "" H 3975 3800 50  0000 C CNN
@@
 $EndComp
 $Comp
-L GND #PWR023
+L GND #PWR013
 U 1 1 5875305D
 P 2875 2650
-F 0 "#PWR023" H 2875 2400 50  0001 C CNN
+F 0 "#PWR013" H 2875 2400 50  0001 C CNN
 F 1 "GND" H 2875 2500 50  0000 C CNN
 F 2 "" H 2875 2650 50  0000 C CNN
@@
 $EndComp
 $Comp
-L +5V #PWR024
+L +5V #PWR014
 U 1 1 58753063
 P 3275 1775
-F 0 "#PWR024" H 3275 1625 50  0001 C CNN
+F 0 "#PWR014" H 3275 1625 50  0001 C CNN
 F 1 "+5V" H 3275 1915 50  0000 C CNN
 F 2 "" H 3275 1775 50  0000 C CNN
@@
 $EndComp
 $Comp
-L GND #PWR025
+L GND #PWR015
 U 1 1 58753070
 P 3525 2775
-F 0 "#PWR025" H 3525 2525 50  0001 C CNN
+F 0 "#PWR015" H 3525 2525 50  0001 C CNN
 F 1 "GND" H 3525 2625 50  0000 C CNN
 F 2 "" H 3525 2775 50  0000 C CNN
@@
 $EndComp
 Wire Wire Line
-	5175 1725 5175 1875
-Connection ~ 5175 1775
-Wire Wire Line
 	5275 5900 5275 5875
 Wire Wire Line
@@
 Wire Wire Line
 	5125 5900 5125 5950
-Connection ~ 5125 5900
 Connection ~ 3275 2175
 Wire Wire Line
@@
 Connection ~ 3650 2725
 Wire Wire Line
-	2900 4000 3500 4000
-Connection ~ 3200 4000
-Wire Wire Line
-	2900 3700 3500 3700
-Connection ~ 3200 3700
-Wire Wire Line
-	2900 4050 2900 4000
-Wire Wire Line
-	2900 3650 2900 3700
-$Comp
-L +5V #PWR026
+	2400 5675 2400 5600
+Wire Wire Line
+	2400 5225 2400 5300
+$Comp
+L +5V #PWR016
 U 1 1 587530B7
 P 5175 1725
-F 0 "#PWR026" H 5175 1575 50  0001 C CNN
+F 0 "#PWR016" H 5175 1575 50  0001 C CNN
 F 1 "+5V" H 5175 1865 50  0000 C CNN
 F 2 "" H 5175 1725 50  0000 C CNN
@@
 	1    0    0    -1
 $EndComp
-$Comp
-L GND #PWR027
-U 1 1 587530BD
-P 5750 1825
-F 0 "#PWR027" H 5750 1575 50  0001 C CNN
-F 1 "GND" H 5750 1675 50  0000 C CNN
-F 2 "" H 5750 1825 50  0000 C CNN
-F 3 "" H 5750 1825 50  0000 C CNN
-	1    5750 1825
-	1    0    0    -1
-$EndComp
-Wire Wire Line
-	5750 1825 5750 1775
 Wire Wire Line
 	6975 4575 6975 4525
@@
 	7825 4675 7725 4675
 Connection ~ 7725 4675
-Wire Wire Line
-	4975 1775 5450 1775
-Wire Wire Line
-	5375 1875 5375 1775
-Connection ~ 5375 1775
-Wire Wire Line
-	4975 5900 5275 5900
 Wire Wire Line
 	2875 2650 2875 2600
@@
 Wire Wire Line
 	3550 3375 4275 3375
-$Comp
-L ATMEGA1284P-A IC1
-U 1 1 588516E2
-P 5275 3875
-F 0 "IC1" H 4425 5755 50  0000 L BNN
-F 1 "ATMEGA1284P-A" H 5675 1925 50  0000 L BNN
-F 2 "Housings_QFP:TQFP-44_10x10mm_Pitch0.8mm" H 5275 3875 50  0001 C CIN
-F 3 "" H 5275 3875 50  0000 C CNN
-	1    5275 3875
-	1    0    0    -1
-$EndComp
 Wire Wire Line
 	5075 1875 5075 1775
-Wire Wire Line
-	4975 1875 4975 1775
-Connection ~ 5075 1775
-Wire Wire Line
-	5175 5875 5175 5900
-Connection ~ 5175 5900
-Wire Wire Line
-	4975 5900 4975 5875
-Connection ~ 5075 5900
 $Comp
 L button-touch-6x6mm SW1
@@
 Connection ~ 2875 2650
 $Comp
-L PWR_FLAG #FLG028
+L PWR_FLAG #FLG017
 U 1 1 587FC76C
 P 3600 3350
-F 0 "#FLG028" H 3600 3445 50  0001 C CNN
+F 0 "#FLG017" H 3600 3445 50  0001 C CNN
 F 1 "PWR_FLAG" H 3600 3530 50  0000 C CNN
 F 2 "" H 3600 3350 50  0000 C CNN
@@
 	3600 3375 3600 3350
 Connection ~ 3600 3375
+Wire Wire Line
+	5275 1775 5275 1875
+Wire Wire Line
+	5175 1775 5175 1725
+Connection ~ 5175 1775
+Wire Wire Line
+	5075 5900 5275 5900
+Connection ~ 5125 5900
+$Comp
+L ATMEGA1284P-P IC1
+U 1 1 58B70CC5
+P 5275 3875
+F 0 "IC1" H 4425 5755 50  0000 L BNN
+F 1 "ATMEGA1284P-P" H 5675 1925 50  0000 L BNN
+F 2 "Housings_DIP:DIP-40_W15.24mm_LongPads" H 5275 3875 50  0000 C CIN
+F 3 "" H 5275 3875 50  0000 C CNN
+	1    5275 3875
+	1    0    0    -1
+$EndComp
+Wire Wire Line
+	5075 1775 5275 1775
+Wire Wire Line
+	2700 5300 2700 5275
+Wire Wire Line
+	2700 5275 2400 5275
+Connection ~ 2400 5275
+Wire Wire Line
+	2700 5600 2700 5625
+Wire Wire Line
+	2700 5625 2400 5625
+Connection ~ 2400 5625
+Text Notes 7950 4550 0    60   ~ 0
+Vérifier si on peut trouver un quartz avec condensateur 6pF dans ce cas pas besoin de C externe
 $EndSCHEMATC
