File: Hardware/digital/kicad/power_supply.sch (KiCad schematic (older format))
At the start: 32 parts, among them P12 CONN_01X02, P13 CONN_01X02, Q2 FQB22P10, Q3 FQB22P10, U6 LM3485, U7 LM1085IS-3.3/NOPB, U8 LM358

Commit message: move to digital 1.1.1
Parts:
- removed C21: 1nF, Capacitors_ThroughHole:C_Rect_L7_W2.5_P5, symbol C
- removed C23, C33: 120uF, Capacitors_ThroughHole:C_Radial_D6.3_L11.2_P2.5, symbol CP
- removed D10: SR5100, Diodes_ThroughHole:Diode_DO-35_SOD27_Horizontal_RM10, symbol D
- removed D4, D5, D6, D7, D8, D9: EGP20A, Diodes_ThroughHole:Diode_DO-35_SOD27_Horizontal_RM10, symbol D
- removed L1: L_Double, digital:DRQ_127, symbol L_Double
- removed P12, P13: CONN_01X02, Pin_Headers:Pin_Header_Straight_1x02, symbol CONN_01X02
- removed Q2, Q3: FQB22P10, digital:D2PAK_2pins, symbol Q_PMOS_GDS
- removed R10: 0.02, Discret:R4-LARGE_PADS, symbol R
- removed R11: 30.1k, Discret:R3-LARGE_PADS, symbol R
- removed R12: 10k, Discret:R3-LARGE_PADS, symbol R
- removed R17: 100k, Discret:R3-LARGE_PADS, symbol R
- removed R9: 82.5k, Discret:R3-LARGE_PADS, symbol R
- removed U6: LM3485, Housings_SSOP:MSOP-8_3x3mm_Pitch0.65mm, symbol LM3485
- removed U7: LM1085IS-3.3/NOPB, digital:D2PAK_3pins, symbol LM1084IS-3.3/NOPB
- added C10: 1u, Capacitors_ThroughHole:C_Radial_D5_L6_P2.5, symbol CP
- added C13: 10n, Capacitors_ThroughHole:C_Rect_L7_W2.5_P5, symbol C_Small
- added C14, C15: 120u, digital:condensator_horizontal_8_11_5, symbol CP
- added D3, D4, D5, D6, D7: SR5100, digital:Diode_DO-27_Horizontal_RM12, symbol D_Schottky
- added D9: BZX79-C4V7,113, Diodes_ThroughHole:Diode_DO-35_SOD27_Horizontal_RM10, symbol ZENER
- added L1: 47u, digital:inductance_murata_1200LRS, symbol INDUCTOR_SMALL
- added P2: CONN_01X03, Pin_Headers:Pin_Header_Angled_1x03, symbol CONN_01X03
- added Q2: NDT2955, TO_SOT_Packages_SMD:SOT-223, symbol Q_PMOS_GDSD
- added S1, S2, S3, S4: CONN_SOLDERABLE, digital:CONN_SOLDERABLE, symbol CONN_01X02
- added U2: MCP1700, TO_SOT_Packages_THT:TO-92_Horizontal1_Inline_Narrow_Oval, symbol MCP1700
- added U7: LM2672M-5.0, Housings_SOIC:SOIC-8_3.9x4.9mm_Pitch1.27mm, symbol LM2672M-5.0
- added W1: Vin, Measurement_Points:Measurement_Point_Square-TH_Big, symbol TEST_1P
- added W2: USBVCC, Measurement_Points:Measurement_Point_Square-TH_Big, symbol TEST_1P
- added W3: +5V, Measurement_Points:Measurement_Point_Square-TH_Big, symbol TEST_1P
- added W4: +3.3V, Measurement_Points:Measurement_Point_Square-TH_Big, symbol TEST_1P
- added W5: +BATT, Measurement_Points:Measurement_Point_Square-TH_Big, symbol TEST_1P
- added W6: GNDPWR, Measurement_Points:Measurement_Point_Square-TH_Big, symbol TEST_1P
- added W7: GND, Measurement_Points:Measurement_Point_Square-TH_Big, symbol TEST_1P
- C11: renamed from C25; value 120uF -> 1u; footprint Capacitors_ThroughHole:C_Radial_D6.3_L11.2_P2.5 -> Capacitors_ThroughHole:C_Radial_D5_L6_P2.5
- C12: renamed from C26; value 100nF -> 100n
- C16: renamed from C32; value 120uF -> 120u; footprint Capacitors_ThroughHole:C_Radial_D6.3_L11.2_P2.5 -> digital:condensator_horizontal_8_11_5
- C17: renamed from C27; value 120uF -> 120u; footprint Capacitors_ThroughHole:C_Radial_D6.3_L11.2_P2.5 -> digital:condensator_horizontal_8_11_5
- C22: value 270pF -> 100n; footprint Capacitors_ThroughHole:C_Rect_L4_W2.5_P2.5 -> Capacitors_ThroughHole:C_Rect_L7_W2.5_P5
- D8: renamed from D11; footprint Diodes_ThroughHole:Diode_DO-35_SOD27_Horizontal_RM10 -> digital:Diode_DO-27_Horizontal_RM12
- R10: renamed from R16; value 100k -> 10k; footprint Discret:R3-LARGE_PADS -> Resistors_ThroughHole:Resistor_Horizontal_RM10mm
- U8: footprint Housings_DIP:DIP-8_W7.62mm_LongPads -> Housings_SOIC:SOIC-8_3.9x4.9mm_Pitch1.27mm
- renumbered C1 to C18, C30 to C19
Connections:
- net FB_buck is gone; now on net GND: C22.2
- net +3V3: now also S2.2 (P2); no longer C11.1, C12.1
- net +5V: now also Q2.3 (S), S1.2 (P2); no longer C22.1
- net +BATT: now also C22.1, W5.1
- net GND: now also D9.2 (A), S3.2 (P2), W7.1; no longer C11.2, C12.2
- net UDC: now also P2.3 (P3)
- net USBVCC: now also Q2.2 (D), Q2.4 (D), W2.1
- net Uac_hi: now also D3.2 (A), D6.1 (K)
- net Uac_lo: now also D4.2 (A), D7.1 (K)
- net at U8.6 (-), U8.7: now also Q2.1 (G)
- net at C19.1, R10.2, U8.3 (+): now also D9.1 (K)
- net VIN renamed Vin
- net Vin: now also S4.2 (P2)
- new net: C13.2, U7.1 (CB)
- new net: C13.1, D5.1 (K), L1.1, U7.8 (VSW)
- new net: D3.1 (K), D4.1 (K), P2.1 (P1)
- new net +3V3_PWR: C11.1, C12.1, S2.1 (P1), U2.3 (VO), W4.1
- new net +5V_PWR: C10.1, C15.1, L1.3, S1.1 (P1), U2.2 (VI), U7.4 (FB), W3.1
- new net GNDPWR: C10.2, C11.2, C12.2, C14.2, C15.2, D5.2 (A), D6.2 (A), D7.2 (A), S3.1 (P1), U2.1 (GND), U7.6 (GND), W6.1
- new net Vin_PWR: C14.1, P2.2 (P2), S4.1 (P1), U7.7 (VIN), W1.1
- no-connect marks 1 -> 3
Other:
- note added: "5 to 4.1V, 2 A, mount it when use the GPRS sim 800L module"
- note added: "Auto switch, if if Vin is set, don't use +5V from USB"
- note added: "DC linear regulator for 3.3V supply"
- note added: "DC-DC converter\nVin 8 to 40V\nVout 5V"
- note added: "DESCRIPTION: \nThese jumpers allow the isolation of the feeder.\nTo be used during the test phase."
- note added: "From shield PCB"
- note added: "JUMPER CONNECTORS"
- note added: "Jumper to select :\nUDC or UAC source"
- note added: "TESTING PINS"
- note added: "VERY IMPORTANT: \nThis pins can be used to implement testing probes."
- note removed: "5 to 4.1V, 2 A"
- note removed: "DC-DC converter\nVin 10 to 30V\nVout 5V"
- moved on the sheet: C11, C12, C16, C17, C18, C19, D8, R10, U8A, U8B
